Commit message: Refactor lidar configuration in mir_robot.gazebo.xacro and sick_s300.gazebo.xacro

File: fws_robot_description/gazebo/mir_robot.gazebo.xacro (robot description, xacro)
@@ -11,7 +11,7 @@
       </plugin>
     </gazebo> -->
-    <gazebo reference="lidar_head_link" >
-      <sensor name="lidar_head_link" type="gpu_lidar">
-        <gz_frame_id>lidar_head_link</gz_frame_id>
+    <gazebo reference="front_laser_link" >
+      <sensor name="front_laser_link" type="gpu_lidar">
+        <gz_frame_id>front_laser_link</gz_frame_id>
         <topic>scan</topic>
         <update_rate>30</update_rate>
@@ -36,5 +36,5 @@
             <resolution>0.01</resolution>
           </range>
-          <frame_id>/lidar_head_link</frame_id>
+          <frame_id>/front_laser_link</frame_id>
         </lidar>
         <alwaysOn>ture</alwaysOn>

File: mir_robot/mir_description/urdf/general/sick_s300.gazebo.xacro (robot description, xacro)
@@ -1,43 +1,38 @@
 <?xml version="1.0"?>
 <robot xmlns:xacro="http://ros.org/wiki/xacro">
-	<xacro:include filename="$(find mir_description)/urdf/general/common_properties.urdf.xacro" />
-	<xacro:macro name="sick_s300_gazebo" params="link topic robot_namespace tf_prefix">
-		<gazebo reference="${link}">
-			<xacro:insert_block name="material_black" />
-			<sensor type="ray" name="${link}">
-				<pose>0 0 0 0 0 0</pose>
-				<visualize>false</visualize>
-				<update_rate>12.5</update_rate>
-				<ray>
-					<scan>
-						<horizontal>
-							<samples>541</samples>
-							<resolution>1</resolution>  <!-- has to be 1; actual resolution will be computed from number of samples + min_angle/max_angle -->
-							<min_angle>-2.35619449615</min_angle>
-							<max_angle>2.35619449615</max_angle>
-						</horizontal>
-					</scan>
-					<range>
-						<min>0.05</min>
-						<max>29.0</max>
-						<resolution>0.01</resolution>
-					</range>
-					<noise>
-						<type>gaussian</type>
-						<!-- Noise parameters based on published spec for S300 achieving
-									"+-29mm" accuracy at range < 3m (~0.01 of the range) at
-									1 sigma. -->
-						<mean>0.0</mean>
-						<stddev>0.01</stddev>
-					</noise>
-				</ray>
-				<plugin name="gazebo_ros_${link}_controller" filename="libgazebo_ros_laser.so">
-					<!-- no tf_prefix, plugin always uses a tf_prefix (if none is set it uses robotNamespace) -->
-					<robotNamespace>${robot_namespace}</robotNamespace>
-					<frameName>${tf_prefix}${link}</frameName>
-					<topicName>${topic}</topicName>
-				</plugin>
-			</sensor>
-		</gazebo>
-	</xacro:macro>
+  <!-- LiDAR macro definition with parameters for flexibility -->
+  <xacro:macro name="sick_s300_gazebo" params="link topic robot_namespace tf_prefix">
+    <!-- LiDAR Sensor Configuration for ROS 2 -->
+    <gazebo reference="${link}">
+      <sensor name="${link}" type="gpu_lidar">
+        <gz_frame_id>${link}</gz_frame_id> <!-- Use the provided link for frame ID -->
+        <topic>${topic}</topic> <!-- Use the provided topic for the scan -->
+        <update_rate>12.5</update_rate> <!-- Retained the original update rate -->
+        <lidar>
+          <scan>
+            <horizontal>
+              <samples>541</samples> <!-- Retained the original sample count -->
+              <resolution>1</resolution> <!-- Retained the original resolution -->
+              <min_angle>-2.35619449615</min_angle> <!-- Same min angle as in the original -->
+              <max_angle>2.35619449615</max_angle> <!-- Same max angle as in the original -->
+            </horizontal>
+            <vertical>
+              <samples>1</samples> <!-- Single vertical sample (no vertical scan in the original) -->
+              <resolution>0.1</resolution> <!-- Set a small resolution for vertical scan -->
+              <min_angle>0.0</min_angle> <!-- No vertical range in original -->
+              <max_angle>0.0</max_angle> <!-- No vertical range in original -->
+            </vertical>
+          </scan>
+          <range>
+            <min>0.05</min> <!-- Retained the original min range -->
+            <max>29.0</max> <!-- Retained the original max range -->
+            <resolution>0.01</resolution>
+          </range>
+          <frame_id>${tf_prefix}${link}</frame_id> <!-- Use tf_prefix and link for frame ID -->
+        </lidar>
+        <alwaysOn>true</alwaysOn>
+        <visualize>false</visualize> <!-- Retained visualize as false -->
+      </sensor>
+    </gazebo>
+  </xacro:macro>
 </robot>

File: mir_robot/mir_description/urdf/mir_600/mir_600.gazebo.xacro (robot description, xacro)
@@ -45,6 +45,6 @@
 		<!-- Add Gazebo xacro for the laser scanner to work in Gazebo -->
 		<!-- Please match there macro calls with the sick_s300 xacro calls in the mir_600.urdf.xacro file-->
-		<xacro:sick_s300_gazebo link="front_laser_link" robot_namespace="${robot_namespace_slashed}" topic="f_scan" tf_prefix="${tf_prefix_slashed}"/>
-		<xacro:sick_s300_gazebo link="back_laser_link" robot_namespace="${robot_namespace_slashed}" topic="b_scan" tf_prefix="${tf_prefix_slashed}"/>
+		<xacro:sick_s300_gazebo link="front_laser_link" robot_namespace="${robot_namespace_slashed}" topic="scan" tf_prefix="${tf_prefix_slashed}"/>
+		<xacro:sick_s300_gazebo link="back_laser_link" robot_namespace="${robot_namespace_slashed}" topic="scan" tf_prefix="${tf_prefix_slashed}"/>
 		<!-- Settings for the camera of the robot to work in the simulation environment-->
     	<xacro:gazebo_d435 camera_name="${robot_namespace_underscored}camera" reference_link="camera_link" topics_ns="${robot_namespace_slashed}camera" depth_optical_frame="${tf_prefix_slashed}camera_depth_optical_frame" color_optical_frame="${tf_prefix_slashed}camera_color_optical_frame" infrared1_optical_frame="${tf_prefix_slashed}camera_left_ir_optical_frame" infrared2_optical_frame="${tf_prefix_slashed}camera_right_ir_optical_frame" publish_pointcloud="true"/>
