Commit message: prismatic joints dont work in ROS2 ??

File: mir_robot/mir_description/urdf/mir_600/mir_600_top_lift.urdf.xacro (robot description, xacro)
@@ -28,11 +28,11 @@
 				</material>
 		</gazebo>
-		<joint name="left_lift_joint" type="prismatic">
+		<joint name="left_lift_joint" type="continuous">
 			<origin xyz="0.0 0.0 0.0" rpy="0 0 0" />
 			<parent link="left_lift_bottom" />
 			<child link="left_lift_top" />
 			<dynamics damping="1.0" friction="1.0"/>
-			<limit lower="0.0" upper="0.5" effort="1000000" velocity="1.0"/>
-			<axis xyz="0 0 1" />
+			<limit lower="0.0" upper="1.0" effort="1000000" velocity="1.0"/>
+			<axis xyz="0 1 0" />
 			<gazebo>
 				<plugin filename="gz_ros2_control-system" name="gz_ros2_control::GazeboSimROS2ControlPlugin"/>

Commit message: Update joint limit parameters for mur_620 robot

File: mir_robot/mir_description/urdf/mir_600/mir_600_top_lift.urdf.xacro (robot description, xacro)
@@ -28,4 +28,5 @@
 				</material>
 		</gazebo>
+		<!-- for some reason prismatic joint dont work, so we use a continuous joint - this is a workaround and should be fixed -->
 		<joint name="left_lift_joint" type="continuous">
 			<origin xyz="0.0 0.0 0.0" rpy="0 0 0" />
@@ -33,5 +34,5 @@
 			<child link="left_lift_top" />
 			<dynamics damping="1.0" friction="1.0"/>
-			<limit lower="0.0" upper="1.0" effort="1000000" velocity="1.0"/>
+			<limit lower="-0.01" upper="1.0" effort="1000000" velocity="1.0"/>
 			<axis xyz="0 1 0" />
 			<gazebo>
@@ -66,10 +67,10 @@
 				</material>
 		</gazebo>
-		<joint name="right_lift_joint" type="prismatic">
+		<joint name="right_lift_joint" type="continuous">
 			<origin xyz="0.0 0.0 0.0" rpy="0 0 0" />
 			<parent link="right_lift_bottom" />
 			<child link="right_lift_top" />
 			<dynamics damping="1.0" friction="1.0"/>
-			<limit lower="0.0" upper="0.5" effort="1000000" velocity="1.0"/>
+			<limit lower="-0.01" upper="0.5" effort="1000000" velocity="1.0"/>
 			<axis xyz="0 0 1" />
 			<gazebo>

File: mir_robot/mir_description/urdf/mur_620.gazebo.xacro (robot description, xacro)
@@ -17,5 +17,5 @@
 	<!-- UR parameters -->
 	<xacro:arg name="ur_type" default="ur10e"/>
-	<xacro:arg name="joint_limit_params" default="$(find mur_moveit_config)/config/joint_limits_ur.yaml"/>
+	<xacro:arg name="joint_limit_params" default="$(find mur_moveit_config)/config/joint_limits.yaml"/>
 	<xacro:arg name="kinematics_params" default="$(find ur_description)/config/$(arg ur_type)/default_kinematics.yaml"/>
 	<xacro:arg name="physical_params" default="$(find ur_description)/config/$(arg ur_type)/physical_parameters.yaml"/>
