Commit message: feat: update odometry parameters and enhance collision properties for wheels

File: mir_robot/mir_description/urdf/mir_600/mir_600_wheels.gazebo.xacro (robot description, xacro)
@@ -9,4 +9,20 @@
 					<emissive>0 0 0 1</emissive>
 				</material>
+				<collision>
+					<surface>
+						<contact>
+							<ode>
+								<kp>1000.0</kp>
+								<kd>5.0</kd>
+							</ode>
+						</contact>
+						<friction>
+							<ode>
+								<mu>10000.0</mu>
+								<mu2>100.0</mu2>
+							</ode>
+						</friction>
+					</surface>
+				</collision>
 		</gazebo>
 	</xacro:macro>
@@ -27,4 +43,20 @@
 					<emissive>0 0 0 1</emissive>
 				</material>
+				<collision>
+					<surface>
+						<contact>
+							<ode>
+								<kp>1000000.0</kp>
+								<kd>0.0</kd>
+							</ode>
+						</contact>
+						<friction>
+							<ode>
+								<mu>0.0</mu>
+								<mu2>0.0</mu2>
+							</ode>
+						</friction>
+					</surface>
+				</collision>
 		</gazebo>
 	</xacro:macro>

Commit message: moveit

File: mir_robot/mir_description/urdf/mir_600/mir_600_wheels.gazebo.xacro (robot description, xacro)
@@ -9,4 +9,20 @@
 					<emissive>0 0 0 1</emissive>
 				</material>
+				<collision>
+					<surface>
+						<contact>
+							<ode>
+								<kp>1000000.0</kp>
+								<kd>1.0</kd>
+							</ode>
+						</contact>
+						<friction>
+							<ode>
+								<mu>200.0</mu>
+								<mu2>200.0</mu2>
+							</ode>
+						</friction>
+					</surface>
+				</collision>
 		</gazebo>
 	</xacro:macro>
@@ -27,4 +43,20 @@
 					<emissive>0 0 0 1</emissive>
 				</material>
+				<collision>
+					<surface>
+						<contact>
+							<ode>
+								<kp>1000000.0</kp>
+								<kd>0.0</kd>
+							</ode>
+						</contact>
+						<friction>
+							<ode>
+								<mu>0.0</mu>
+								<mu2>0.0</mu2>
+							</ode>
+						</friction>
+					</surface>
+				</collision>
 		</gazebo>
 	</xacro:macro>
