Commit message: feat: Update caster wheel visuals to support high-quality options and simplify mesh usage

File: mir_robot/mir_description/urdf/mir_600/mir_600.urdf.xacro (robot description, xacro)
@@ -125,8 +125,8 @@
 		<xacro:actuated_wheel locationprefix="left" locationright="-1" use_simple_visuals="${use_simple_visuals}" use_wheel_visual_mesh="${use_wheel_visual_mesh}"/>
 		<xacro:actuated_wheel locationprefix="right" locationright="1" use_simple_visuals="${use_simple_visuals}" use_wheel_visual_mesh="${use_wheel_visual_mesh}"/>
-		<xacro:caster_wheel locationprefix="fl" locationright="-1" wheel_base_dx="${mir_600_front_caster_wheel_base_dx}" use_simple_collisions="${use_simple_collisions}" use_simple_visuals="${use_simple_visuals}" use_caster_visual_mesh="${use_caster_visual_mesh}"/>
-		<xacro:caster_wheel locationprefix="fr" locationright="1" wheel_base_dx="${mir_600_front_caster_wheel_base_dx}" use_simple_collisions="${use_simple_collisions}" use_simple_visuals="${use_simple_visuals}" use_caster_visual_mesh="${use_caster_visual_mesh}"/>
-		<xacro:caster_wheel locationprefix="bl" locationright="-1" wheel_base_dx="${mir_600_back_caster_wheel_base_dx}" use_simple_collisions="${use_simple_collisions}" use_simple_visuals="${use_simple_visuals}" use_caster_visual_mesh="${use_caster_visual_mesh}"/>
-		<xacro:caster_wheel locationprefix="br" locationright="1" wheel_base_dx="${mir_600_back_caster_wheel_base_dx}" use_simple_collisions="${use_simple_collisions}" use_simple_visuals="${use_simple_visuals}" use_caster_visual_mesh="${use_caster_visual_mesh}"/>
+		<xacro:caster_wheel locationprefix="fl" locationright="-1" wheel_base_dx="${mir_600_front_caster_wheel_base_dx}" use_simple_collisions="${use_simple_collisions}" use_simple_visuals="${use_simple_visuals}" use_high_quality_visuals="${use_high_quality_visuals}" use_caster_visual_mesh="${use_caster_visual_mesh}"/>
+		<xacro:caster_wheel locationprefix="fr" locationright="1" wheel_base_dx="${mir_600_front_caster_wheel_base_dx}" use_simple_collisions="${use_simple_collisions}" use_simple_visuals="${use_simple_visuals}" use_high_quality_visuals="${use_high_quality_visuals}" use_caster_visual_mesh="${use_caster_visual_mesh}"/>
+		<xacro:caster_wheel locationprefix="bl" locationright="-1" wheel_base_dx="${mir_600_back_caster_wheel_base_dx}" use_simple_collisions="${use_simple_collisions}" use_simple_visuals="${use_simple_visuals}" use_high_quality_visuals="${use_high_quality_visuals}" use_caster_visual_mesh="${use_caster_visual_mesh}"/>
+		<xacro:caster_wheel locationprefix="br" locationright="1" wheel_base_dx="${mir_600_back_caster_wheel_base_dx}" use_simple_collisions="${use_simple_collisions}" use_simple_visuals="${use_simple_visuals}" use_high_quality_visuals="${use_high_quality_visuals}" use_caster_visual_mesh="${use_caster_visual_mesh}"/>
 		<joint name="base_link_surface_joint" type="fixed">
 			<origin xyz="${mir_600_act_wheel_dx} 0 0.352" rpy="0 0 0" />

File: mir_robot/mir_description/urdf/mir_600/mir_600_wheels.urdf.xacro (robot description, xacro)
@@ -40,5 +40,5 @@
 		</link>
 	</xacro:macro>
-	<xacro:macro name="caster_wheel" params="locationprefix locationright wheel_base_dx use_simple_collisions:=false use_simple_visuals:=false use_caster_visual_mesh:=false">
+	<xacro:macro name="caster_wheel" params="locationprefix locationright wheel_base_dx use_simple_collisions:=false use_simple_visuals:=false use_high_quality_visuals:=false use_caster_visual_mesh:=false">
 		<!-- caster hub -->
 		<joint name="${locationprefix}_caster_rotation_joint" type="continuous">
@@ -121,5 +121,10 @@
 					<origin xyz="0 0 0" rpy="${pi * 0.5} 0 0" />
 					<geometry>
-						<mesh filename="package://mir_description/meshes/visual/mir_600_caster_wheel.stl" />
+						<xacro:if value="${use_high_quality_visuals}">
+							<mesh filename="package://mir_description/meshes/visual/mir_600_caster_wheel.stl" />
+						</xacro:if>
+						<xacro:unless value="${use_high_quality_visuals}">
+							<mesh filename="package://mir_description/meshes/visual/simplify_caster_wheel_mir600.stl" />
+						</xacro:unless>
 					</geometry>
 					<xacro:insert_block name="material_dark_grey" />

Commit message: feat: Add support for MiR 600 variant and enhance robot state publishing

File: mir_robot/mir_description/urdf/mir_600/mir_600.urdf.xacro (robot description, xacro)
@@ -96,4 +96,11 @@
 		</joint>
 		<link name="imu_frame" />
+		<!-- Virtual link for the merged laser scan. -->
+		<joint name="base_link_to_virtual_laser_joint" type="fixed">
+			<parent link="base_link" />
+			<child link="virtual_laser_link" />
+			<origin xyz="0.0 0.0 0.25" rpy="0.0 0.0 0" />
+		</joint>
+		<link name="virtual_laser_link" />
 		<!-- Laser scanners -->
 		<joint name="base_link_to_front_laser_joint" type="fixed">
