Commit message: navigation improvements

File: mir_robot/mir_description/urdf/general/mir.ros2_control.xacro (robot description, xacro)
@@ -7,6 +7,6 @@
     <joint name="left_wheel_joint">
       <command_interface name="velocity">
-        <param name="min">-1</param>
-        <param name="max">1</param>
+        <param name="min">-12</param>
+        <param name="max">12</param>
       </command_interface>
       <state_interface name="position"/>
@@ -15,6 +15,6 @@
     <joint name="right_wheel_joint">
       <command_interface name="velocity">
-        <param name="min">-1</param>
-        <param name="max">1</param>
+        <param name="min">-12</param>
+        <param name="max">12</param>
       </command_interface>
       <state_interface name="position"/>
@@ -29,6 +29,6 @@
       <joint name="left_wheel_joint">
         <command_interface name="velocity">
-          <param name="min">-1</param>
-          <param name="max">1</param>
+          <param name="min">-12</param>
+          <param name="max">12</param>
         </command_interface>
         <state_interface name="position"/>
@@ -38,6 +38,6 @@
       <joint name="right_wheel_joint">
         <command_interface name="velocity">
-          <param name="min">-1</param>
-          <param name="max">1</param>
+          <param name="min">-12</param>
+          <param name="max">12</param>
         </command_interface>
         <state_interface name="position"/>

File: mir_robot/mir_description/urdf/mir_600/mir_600_wheels.gazebo.xacro (robot description, xacro)
@@ -9,20 +9,4 @@
 					<emissive>0 0 0 1</emissive>
 				</material>
-				<collision>
-					<surface>
-						<contact>
-							<ode>
-								<kp>1000.0</kp>
-								<kd>5.0</kd>
-							</ode>
-						</contact>
-						<friction>
-							<ode>
-								<mu>10000.0</mu>
-								<mu2>100.0</mu2>
-							</ode>
-						</friction>
-					</surface>
-				</collision>
 		</gazebo>
 	</xacro:macro>
@@ -43,20 +27,4 @@
 					<emissive>0 0 0 1</emissive>
 				</material>
-				<collision>
-					<surface>
-						<contact>
-							<ode>
-								<kp>1000000.0</kp>
-								<kd>0.0</kd>
-							</ode>
-						</contact>
-						<friction>
-							<ode>
-								<mu>0.0</mu>
-								<mu2>0.0</mu2>
-							</ode>
-						</friction>
-					</surface>
-				</collision>
 		</gazebo>
 	</xacro:macro>
