Commit message: Refactor URDF and launch files for MiR600 and Mur620
- Updated URDF files for MiR600 to include parameters for camera and collision handling.
- Modified top lift and top module URDFs to support simple collision geometries.
- Enhanced caster wheel URDF to allow for simple collision options.
- Added support for camera and arms in Mur620 launch files with appropriate parameters.
- Introduced new RViz configuration for multi-base visualization.
- Updated launch scripts to include new parameters and improved organization.
- Changed default launch behavior to use multi_mur_base.launch.py.

File: mir_robot/mir_description/urdf/general/sick_s300.urdf.xacro (robot description, xacro)
@@ -6,5 +6,5 @@
 	<xacro:property name="laser_z" value="0.185" />
 	<xacro:property name="laser_mass" value="2.0" />
-	<xacro:macro name="sick_s300" params="link topic">
+	<xacro:macro name="sick_s300" params="link topic use_simple_collisions:=false">
 		<link name="${link}">
 			<visual>
@@ -16,10 +16,20 @@
 				<xacro:insert_block name="material_black" />
 			</visual>
-			<collision>
-				<origin xyz="0.0 0.0 0.0" rpy="${pi} 0 0" />
-				<geometry>
-					<mesh filename="package://mir_description/meshes/visual/sick_lms-100.stl" />
-				</geometry>
-			</collision>
+			<xacro:if value="${use_simple_collisions}">
+				<collision>
+					<origin xyz="0.0 0.0 0.0" rpy="0 0 0" />
+					<geometry>
+						<box size="${laser_x} ${laser_y} ${laser_z}"/>
+					</geometry>
+				</collision>
+			</xacro:if>
+			<xacro:unless value="${use_simple_collisions}">
+				<collision>
+					<origin xyz="0.0 0.0 0.0" rpy="${pi} 0 0" />
+					<geometry>
+						<mesh filename="package://mir_description/meshes/visual/sick_lms-100.stl" />
+					</geometry>
+				</collision>
+			</xacro:unless>
 			<xacro:box_inertial x="${laser_x}" y="${laser_y}" z="${laser_z}" mass="${laser_mass}">
 				<origin xyz="0 0 0" />

File: mir_robot/mir_description/urdf/mir_600/mir_600.gazebo.xacro (robot description, xacro)
@@ -8,5 +8,5 @@
 	<xacro:include filename="$(find mir_description)/urdf/general/_d435.gazebo.xacro" />
 	<xacro:property name="imu_standard_deviation" value="0.00017" />
-	<xacro:macro name="mir_600_gazebo" params="tf_prefix robot_namespace">
+	<xacro:macro name="mir_600_gazebo" params="tf_prefix robot_namespace use_camera:=true">
 		<!-- Predefine some values that are necessary later. It is important to differenciate between empty and not empty robot_namespace and tf_prefix -->
 		<xacro:if value="${robot_namespace == ''}">
@@ -46,12 +46,12 @@
 		<!-- Add transmissions to wheels -->
 		<xacro:mir_600_wheel_transmissions/>
-		<!-- Settings for the IMU of the robot to work in the simulation environment-->
-		<xacro:imu_gazebo link="imu_link" robot_namespace="${robot_namespace_slashed}" imu_topic="imu_data" update_rate="50.0" standard_deviation="${imu_standard_deviation}" />
 		<!-- Add Gazebo xacro for the laser scanner to work in Gazebo -->
 		<!-- Please match there macro calls with the sick_s300 xacro calls in the mir_600.urdf.xacro file-->
 		<xacro:sick_s300_gazebo link="front_laser_link" robot_namespace="${robot_namespace_slashed}" topic="${tf_prefix_slashed}f_scan" tf_prefix="${tf_prefix_slashed}"/>
 		<xacro:sick_s300_gazebo link="back_laser_link" robot_namespace="${robot_namespace_slashed}" topic="${tf_prefix_slashed}b_scan" tf_prefix="${tf_prefix_slashed}"/>
-		<!-- Settings for the camera of the robot to work in the simulation environment-->
-    	<xacro:gazebo_d435 camera_name="${robot_namespace_underscored}camera" reference_link="camera_link" topics_ns="${robot_namespace_slashed}camera" depth_optical_frame="${tf_prefix_slashed}camera_depth_optical_frame" color_optical_frame="${tf_prefix_slashed}camera_color_optical_frame" infrared1_optical_frame="${tf_prefix_slashed}camera_left_ir_optical_frame" infrared2_optical_frame="${tf_prefix_slashed}camera_right_ir_optical_frame" publish_pointcloud="true"/>
+		<xacro:if value="${use_camera}">
+			<!-- Settings for the camera of the robot to work in the simulation environment-->
+			<xacro:gazebo_d435 camera_name="${robot_namespace_underscored}camera" reference_link="camera_link" topics_ns="${robot_namespace_slashed}camera" depth_optical_frame="${tf_prefix_slashed}camera_depth_optical_frame" color_optical_frame="${tf_prefix_slashed}camera_color_optical_frame" infrared1_optical_frame="${tf_prefix_slashed}camera_left_ir_optical_frame" infrared2_optical_frame="${tf_prefix_slashed}camera_right_ir_optical_frame" publish_pointcloud="true"/>
+		</xacro:if>
 		<!-- disabled, because it doesn't make a difference in Gazebo: -->
 		<!-- <xacro:set_all_wheel_frictions tf_prefix="${tf_prefix}"/> -->

File: mir_robot/mir_description/urdf/mir_600/mir_600.urdf.xacro (robot description, xacro)
@@ -29,5 +29,5 @@
 	<xacro:property name="mir_600_match_logo_dy" value="0.330" />
 	<xacro:property name="mir_600_match_logo_dz" value="0.27" />
-	<xacro:macro name="mir_600">
+	<xacro:macro name="mir_600" params="use_camera:=true use_simple_collisions:=false">
 		<link name="base_footprint" />
 		<joint name="base_joint" type="fixed">
@@ -47,10 +47,20 @@
 				<xacro:insert_block name="material_white" />
 			</visual>
-			<collision>
-				<origin xyz="${mir_600_act_wheel_dx} 0 0" rpy="${pi * 0.5} 0 ${pi * 0.5}" />
-				<geometry>
-					<mesh filename="package://mir_description/meshes/collision/mir_600_base.stl"/>
-				</geometry>
-			</collision>
+			<xacro:if value="${use_simple_collisions}">
+				<collision>
+					<origin xyz="${mir_600_act_wheel_dx} 0 0.20" rpy="0 0 0" />
+					<geometry>
+						<box size="0.9 0.58 0.3"/>
+					</geometry>
+				</collision>
+			</xacro:if>
+			<xacro:unless value="${use_simple_collisions}">
+				<collision>
+					<origin xyz="${mir_600_act_wheel_dx} 0 0" rpy="${pi * 0.5} 0 ${pi * 0.5}" />
+					<geometry>
+						<mesh filename="package://mir_description/meshes/collision/mir_600_base.stl"/>
+					</geometry>
+				</collision>
+			</xacro:unless>
 		</link>
 		<!-- IMU -->
@@ -76,5 +86,5 @@
 			<origin xyz="0.58985 0.370 0.1914" rpy="0.0 0.0 ${0.25 * pi}" />  <!-- from visually matching up the meshes of the MiR and the laser scanner -->
 		</joint>
-		<xacro:sick_s300 link="front_laser_link" topic="f_scan" />
+		<xacro:sick_s300 link="front_laser_link" topic="f_scan" use_simple_collisions="${use_simple_collisions}" />
 		<joint name="base_link_to_back_laser_joint" type="fixed">
 			<parent link="base_link" />
@@ -82,5 +92,5 @@
 			<origin xyz="-0.58985 -0.370 0.1914" rpy="0.0 0.0 ${-0.75 * pi}" />  <!-- from visually matching up the meshes of the MiR and the laser scanner -->
 		</joint>
-		<xacro:sick_s300 link="back_laser_link" topic="b_scan" />
+		<xacro:sick_s300 link="back_laser_link" topic="b_scan" use_simple_collisions="${use_simple_collisions}" />
 		<!-- Ultrasound sensors -->
 		<joint name="us_1_joint" type="fixed">   <!-- right ultrasound -->
@@ -99,8 +109,8 @@
 		<xacro:actuated_wheel locationprefix="left" locationright="-1"/>
 		<xacro:actuated_wheel locationprefix="right" locationright="1"/>
-		<xacro:caster_wheel locationprefix="fl" locationright="-1" wheel_base_dx="${mir_600_front_caster_wheel_base_dx}"/>
-		<xacro:caster_wheel locationprefix="fr" locationright="1" wheel_base_dx="${mir_600_front_caster_wheel_base_dx}"/>
-		<xacro:caster_wheel locationprefix="bl" locationright="-1" wheel_base_dx="${mir_600_back_caster_wheel_base_dx}"/>
-		<xacro:caster_wheel locationprefix="br" locationright="1" wheel_base_dx="${mir_600_back_caster_wheel_base_dx}"/>
+		<xacro:caster_wheel locationprefix="fl" locationright="-1" wheel_base_dx="${mir_600_front_caster_wheel_base_dx}" use_simple_collisions="${use_simple_collisions}"/>
+		<xacro:caster_wheel locationprefix="fr" locationright="1" wheel_base_dx="${mir_600_front_caster_wheel_base_dx}" use_simple_collisions="${use_simple_collisions}"/>
+		<xacro:caster_wheel locationprefix="bl" locationright="-1" wheel_base_dx="${mir_600_back_caster_wheel_base_dx}" use_simple_collisions="${use_simple_collisions}"/>
+		<xacro:caster_wheel locationprefix="br" locationright="1" wheel_base_dx="${mir_600_back_caster_wheel_base_dx}" use_simple_collisions="${use_simple_collisions}"/>
 		<joint name="base_link_surface_joint" type="fixed">
 			<origin xyz="${mir_600_act_wheel_dx} 0 0.352" rpy="0 0 0" />
@@ -110,12 +120,14 @@
 		</joint>
 		<link name="surface"/>
-		<!--Realsense_Intel_D435_Camera-->
-		<xacro:sensor_d435 name="camera" parent="base_link" use_nominal_extrinsics="true">
-    		<origin xyz="0.62335 0 0.24" rpy="0 0 0" />
-  		</xacro:sensor_d435>
+		<xacro:if value="${use_camera}">
+			<!--Realsense_Intel_D435_Camera-->
+			<xacro:sensor_d435 name="camera" parent="base_link" use_nominal_extrinsics="true">
+				<origin xyz="0.62335 0 0.24" rpy="0 0 0" />
+			</xacro:sensor_d435>
+		</xacro:if>
 		<!-- Insert a match logo on both sides of the mobile robot -->
 		<!-- <xacro:match_logo parent="base_link" locationprefix="left" location_dx="${mir_600_match_logo_dx}" location_dy="${mir_600_match_logo_dy}" location_dz="${mir_600_match_logo_dz}"/>
 		<xacro:match_logo parent="base_link" locationprefix="right" location_dx="${mir_600_match_logo_dx}" location_dy="${-1 * mir_600_match_logo_dy}" location_dz="${mir_600_match_logo_dz}" orientation="${pi}"/> -->
-		<xacro:top_module/>
+		<xacro:top_module use_simple_collisions="${use_simple_collisions}"/>
 		<!-- Camera -->
 		<!--link name="camera_link">

File: mir_robot/mir_description/urdf/mir_600/mir_600_top_lift.urdf.xacro (robot description, xacro)
@@ -1,5 +1,5 @@
 <?xml version="1.0"?>
 <robot xmlns:xacro="http://ros.org/wiki/xacro">
-    <xacro:macro name="top_lift" params="">
+    <xacro:macro name="top_lift" params="use_simple_collisions:=false">
         <link name="left_lift_top">
 			<xacro:box_inertial mass="1.0" x="0.2" y="0.2" z="0.3">
@@ -13,10 +13,20 @@
 				<xacro:insert_block name="material_white" />
 			</visual>
-			<collision>
-				<origin xyz="0 0 0" rpy="${pi * 0.5} 0 ${pi * 0.0}" />
-				<geometry>
-					<mesh filename="package://mir_description/meshes/collision/mir_600_lift_top.stl"/>
-				</geometry>
-			</collision>
+			<xacro:if value="${use_simple_collisions}">
+				<collision>
+					<origin xyz="0 0 0.15" rpy="0 0 0" />
+					<geometry>
+						<box size="0.2 0.2 0.3"/>
+					</geometry>
+				</collision>
+			</xacro:if>
+			<xacro:unless value="${use_simple_collisions}">
+				<collision>
+					<origin xyz="0 0 0" rpy="${pi * 0.5} 0 ${pi * 0.0}" />
+					<geometry>
+						<mesh filename="package://mir_description/meshes/collision/mir_600_lift_top.stl"/>
+					</geometry>
+				</collision>
+			</xacro:unless>
 		</link>
 		<gazebo reference="left_lift_top">
@@ -47,10 +57,20 @@
 				<xacro:insert_block name="material_white" />
 			</visual>
-			<collision>
-				<origin xyz="0 0 0" rpy="${pi * 0.5} 0 ${pi * 0.0}" />
-				<geometry>
-					<mesh filename="package://mir_description/meshes/collision/mir_600_lift_top.stl"/>
-				</geometry>
-			</collision>
+			<xacro:if value="${use_simple_collisions}">
+				<collision>
+					<origin xyz="0 0 0.15" rpy="0 0 0" />
+					<geometry>
+						<box size="0.2 0.2 0.3"/>
+					</geometry>
+				</collision>
+			</xacro:if>
+			<xacro:unless value="${use_simple_collisions}">
+				<collision>
+					<origin xyz="0 0 0" rpy="${pi * 0.5} 0 ${pi * 0.0}" />
+					<geometry>
+						<mesh filename="package://mir_description/meshes/collision/mir_600_lift_top.stl"/>
+					</geometry>
+				</collision>
+			</xacro:unless>
 		</link>
 		<gazebo reference="right_lift_top">

File: mir_robot/mir_description/urdf/mir_600/mir_600_top_module.urdf.xacro (robot description, xacro)
@@ -2,5 +2,5 @@
 <robot xmlns:xacro="http://ros.org/wiki/xacro">
 	<xacro:include filename="$(find mir_description)/urdf/general/common_properties.urdf.xacro" />
-	<xacro:macro name="top_module" params="">
+	<xacro:macro name="top_module" params="use_simple_collisions:=false">
 		<!-- top module -->
 		<link name="top_module">
@@ -47,10 +47,20 @@
 				<xacro:insert_block name="material_white" />
 			</visual>
-			<collision>
-				<origin xyz="0 0 0" rpy="${pi * 0.5} 0 ${pi * 0.0}" />
-				<geometry>
-					<mesh filename="package://mir_description/meshes/collision/mir_600_lift_bot.stl"/>
-				</geometry>
-			</collision>
+			<xacro:if value="${use_simple_collisions}">
+				<collision>
+					<origin xyz="0 0 0.15" rpy="0 0 0" />
+					<geometry>
+						<box size="0.2 0.2 0.3"/>
+					</geometry>
+				</collision>
+			</xacro:if>
+			<xacro:unless value="${use_simple_collisions}">
+				<collision>
+					<origin xyz="0 0 0" rpy="${pi * 0.5} 0 ${pi * 0.0}" />
+					<geometry>
+						<mesh filename="package://mir_description/meshes/collision/mir_600_lift_bot.stl"/>
+					</geometry>
+				</collision>
+			</xacro:unless>
 		</link>
 		<gazebo reference="left_lift_bottom">
@@ -79,10 +89,20 @@
 				<xacro:insert_block name="material_white" />
 			</visual>
-			<collision>
-				<origin xyz="0 0 0" rpy="${pi * 0.5} 0 ${pi * 0.0}" />
-				<geometry>
-					<mesh filename="package://mir_description/meshes/collision/mir_600_lift_bot.stl"/>
-				</geometry>
-			</collision>
+			<xacro:if value="${use_simple_collisions}">
+				<collision>
+					<origin xyz="0 0 0.15" rpy="0 0 0" />
+					<geometry>
+						<box size="0.2 0.2 0.3"/>
+					</geometry>
+				</collision>
+			</xacro:if>
+			<xacro:unless value="${use_simple_collisions}">
+				<collision>
+					<origin xyz="0 0 0" rpy="${pi * 0.5} 0 ${pi * 0.0}" />
+					<geometry>
+						<mesh filename="package://mir_description/meshes/collision/mir_600_lift_bot.stl"/>
+					</geometry>
+				</collision>
+			</xacro:unless>
 		</link>
 		<gazebo reference="right_lift_bottom">

File: mir_robot/mir_description/urdf/mir_600/mir_600_wheels.urdf.xacro (robot description, xacro)
@@ -29,5 +29,5 @@
 		</link>
 	</xacro:macro>
-	<xacro:macro name="caster_wheel" params="locationprefix locationright wheel_base_dx">
+	<xacro:macro name="caster_wheel" params="locationprefix locationright wheel_base_dx use_simple_collisions:=false">
 		<!-- caster hub -->
 		<joint name="${locationprefix}_caster_rotation_joint" type="continuous">
@@ -58,10 +58,20 @@
 			<xacro:insert_block name="material_silver" />
 		</visual>
-		<collision>
-			<origin xyz="0 0 0" rpy="0 0 0" />
-			<geometry>
-				<mesh filename="package://mir_description/meshes/collision/caster_wheel_base.stl" />
-			</geometry>
-		</collision>
+		<xacro:if value="${use_simple_collisions}">
+			<collision>
+				<origin xyz="0 0 -0.03" rpy="0 0 0" />
+				<geometry>
+					<box size="0.16 0.12 0.08"/>
+				</geometry>
+			</collision>
+		</xacro:if>
+		<xacro:unless value="${use_simple_collisions}">
+			<collision>
+				<origin xyz="0 0 0" rpy="0 0 0" />
+				<geometry>
+					<mesh filename="package://mir_description/meshes/collision/caster_wheel_base.stl" />
+				</geometry>
+			</collision>
+		</xacro:unless>
 		</link>
 		<!-- caster wheel -->

File: mur_robot/mur_description/urdf/mur_620.gazebo.xacro (robot description, xacro)
@@ -5,4 +5,10 @@
 	<xacro:arg name="tf_prefix_mir" default='mur620'/>
 	<xacro:arg name="name" default=''/>
+	<xacro:arg name="use_arms" default='true'/>
+	<xacro:property name="use_arms" value="$(arg use_arms)"/>
+	<xacro:arg name="use_camera" default='true'/>
+	<xacro:property name="use_camera" value="$(arg use_camera)"/>
+	<xacro:arg name="use_simple_collisions" default='false'/>
+	<xacro:property name="use_simple_collisions" value="$(arg use_simple_collisions)"/>
 	<xacro:arg name="use_lift" default='true'/>
 	<xacro:property name="use_lift" value="$(arg use_lift)"/>
@@ -38,7 +44,10 @@
 	<xacro:include filename="$(find mir_description)/urdf/general/plugins.gazebo.xacro" />
 	<!-- Init the MiR600 marco that is also used for the hardware -->
-	<xacro:mir_600/>
+	<xacro:mir_600
+		use_camera="$(arg use_camera)"
+		use_simple_collisions="$(arg use_simple_collisions)"
+	/>
 	<!-- Init the MiR600 macro that includes all infos that Gazebo need to function -->
-	<xacro:mir_600_gazebo tf_prefix="$(arg tf_prefix_mir)" robot_namespace="$(arg robot_namespace)"/>
+	<xacro:mir_600_gazebo tf_prefix="$(arg tf_prefix_mir)" robot_namespace="$(arg robot_namespace)" use_camera="$(arg use_camera)"/>
 	<!-- Init the plugins that run the MiR in Gazebo -->
 	<xacro:controller_plugin_gazebo
@@ -46,78 +55,83 @@
 		controllers_file="$(arg simulation_controllers)"
 	/>
-	<xacro:p3d_base_controller robot_namespace="$(arg robot_namespace)"/>
 	<xacro:gazebo_sim_sensors robot_namespace="$(arg robot_namespace)"/>
 	<xacro:mir_robot_ros2_control/>
-	<!-- UR10_l -->
-	<xacro:ur_robot
-		name="UR10_l"
-		tf_prefix="UR10_l/"
-		parent="UR10_l/base_ideal"
-		joint_limits_parameters_file="$(arg joint_limit_params)"
-		kinematics_parameters_file="$(arg kinematics_params)"
-		physical_parameters_file="$(arg physical_params)"
-		visual_parameters_file="$(arg visual_params)"
-		safety_limits="$(arg safety_limits)"
-		safety_pos_margin="$(arg safety_pos_margin)"
-		safety_k_position="$(arg safety_k_position)"
-		force_abs_paths="true"
-		>
-		<origin xyz="0 0 0" rpy="$(arg ur_l_rpy)" />          <!-- position robot in the world -->
-  	</xacro:ur_robot>
-	<xacro:ur_robot
-		name="UR10_r"
-		tf_prefix="UR10_r/"
-		parent="UR10_r/base_ideal"
-		joint_limits_parameters_file="$(arg joint_limit_params)"
-		kinematics_parameters_file="$(arg kinematics_params)"
-		physical_parameters_file="$(arg physical_params)"
-		visual_parameters_file="$(arg visual_params)"
-		safety_limits="$(arg safety_limits)"
-		safety_pos_margin="$(arg safety_pos_margin)"
-		safety_k_position="$(arg safety_k_position)"
-		force_abs_paths="true"
-		>
-		<origin xyz="0 0 0" rpy="$(arg ur_r_rpy)" />          <!-- position robot in the world -->
-  	</xacro:ur_robot>
-	<xacro:ur_ros2_control
-		name="UR10_l"
-		tf_prefix="UR10_l/"
-		transmission_hw_interface="$(arg transmission_hw_interface)"
-		initial_positions="${dict(shoulder_pan_joint=0.0,shoulder_lift_joint=-1.57079632679,elbow_joint=-1.57079632679,wrist_1_joint=-1.57079632679,wrist_2_joint=1.57079632679,wrist_3_joint=0.0)}"
-	/>
-	<xacro:ur_ros2_control
-		name="UR10_r"
-		tf_prefix="UR10_r/"
-		transmission_hw_interface="$(arg transmission_hw_interface)"
-		initial_positions="${dict(shoulder_pan_joint=3.14159265359,shoulder_lift_joint=-1.57079632679,elbow_joint=-1.57079632679,wrist_1_joint=-1.57079632679,wrist_2_joint=-1.57079632679,wrist_3_joint=0.0)}"
-	/>
+	<xacro:if value="${use_arms}">
+		<!-- UR10_l -->
+		<xacro:ur_robot
+			name="UR10_l"
+			tf_prefix="UR10_l/"
+			parent="UR10_l/base_ideal"
+			joint_limits_parameters_file="$(arg joint_limit_params)"
+			kinematics_parameters_file="$(arg kinematics_params)"
+			physical_parameters_file="$(arg physical_params)"
+			visual_parameters_file="$(arg visual_params)"
+			safety_limits="$(arg safety_limits)"
+			safety_pos_margin="$(arg safety_pos_margin)"
+			safety_k_position="$(arg safety_k_position)"
+			force_abs_paths="true"
+			>
+			<origin xyz="0 0 0" rpy="$(arg ur_l_rpy)" />          <!-- position robot in the world -->
+		</xacro:ur_robot>
+		<xacro:ur_robot
+			name="UR10_r"
+			tf_prefix="UR10_r/"
+			parent="UR10_r/base_ideal"
+			joint_limits_parameters_file="$(arg joint_limit_params)"
+			kinematics_parameters_file="$(arg kinematics_params)"
+			physical_parameters_file="$(arg physical_params)"
+			visual_parameters_file="$(arg visual_params)"
+			safety_limits="$(arg safety_limits)"
+			safety_pos_margin="$(arg safety_pos_margin)"
+			safety_k_position="$(arg safety_k_position)"
+			force_abs_paths="true"
+			>
+			<origin xyz="0 0 0" rpy="$(arg ur_r_rpy)" />          <!-- position robot in the world -->
+		</xacro:ur_robot>
+		<xacro:ur_ros2_control
+			name="UR10_l"
+			tf_prefix="UR10_l/"
+			transmission_hw_interface="$(arg transmission_hw_interface)"
+			initial_positions="${dict(shoulder_pan_joint=0.0,shoulder_lift_joint=-1.57079632679,elbow_joint=-1.57079632679,wrist_1_joint=-1.57079632679,wrist_2_joint=1.57079632679,wrist_3_joint=0.0)}"
+		/>
+		<xacro:ur_ros2_control
+			name="UR10_r"
+			tf_prefix="UR10_r/"
+			transmission_hw_interface="$(arg transmission_hw_interface)"
+			initial_positions="${dict(shoulder_pan_joint=3.14159265359,shoulder_lift_joint=-1.57079632679,elbow_joint=-1.57079632679,wrist_1_joint=-1.57079632679,wrist_2_joint=-1.57079632679,wrist_3_joint=0.0)}"
+		/>
 		<!-- virtual link rotated to show in same direction like mir  -->
-	<link name="UR10_l/base_ideal" />
-	<link name="UR10_r/base_ideal" />
+		<link name="UR10_l/base_ideal" />
+		<link name="UR10_r/base_ideal" />
+	</xacro:if>
 	<!-- Init the lift macro -->
 	<xacro:if value="${use_lift}">
-		<xacro:top_lift/>
-		<joint name="plattform_manipulator_joint_l" type="fixed">
-				<parent link="left_lift_top" />
+		<xacro:top_lift use_simple_collisions="$(arg use_simple_collisions)"/>
+		<xacro:if value="${use_arms}">
+			<joint name="plattform_manipulator_joint_l" type="fixed">
+					<parent link="left_lift_top" />
+					<child link="UR10_l/base_ideal" />
+					<origin xyz="0.0 0.0 0.555" rpy="0 0 0" />
+			</joint>
+			<joint name="plattform_manipulator_joint_r" type="fixed">
+					<parent link="right_lift_top" />
+					<child link="UR10_r/base_ideal" />
+					<origin xyz="0.0 0.0 0.555" rpy="0 0 0" />
+			</joint>
+		</xacro:if>
+	</xacro:if>
+	<xacro:unless value="${use_lift}">
+		<xacro:if value="${use_arms}">
+			<joint name="plattform_manipulator_joint_l" type="fixed">
+				<parent link="left_lift_bottom" />
 				<child link="UR10_l/base_ideal" />
 				<origin xyz="0.0 0.0 0.555" rpy="0 0 0" />
-		</joint>
-		<joint name="plattform_manipulator_joint_r" type="fixed">
-				<parent link="right_lift_top" />
+			</joint>
+			<joint name="plattform_manipulator_joint_r" type="fixed">
+				<parent link="right_lift_bottom" />
 				<child link="UR10_r/base_ideal" />
 				<origin xyz="0.0 0.0 0.555" rpy="0 0 0" />
-		</joint>
-	</xacro:if>
-	<xacro:unless value="${use_lift}">
-		<joint name="plattform_manipulator_joint_l" type="fixed">
-			<parent link="left_lift_bottom" />
-			<child link="UR10_l/base_ideal" />
-			<origin xyz="0.0 0.0 0.555" rpy="0 0 0" />
-		</joint>
-		<joint name="plattform_manipulator_joint_r" type="fixed">
-			<parent link="right_lift_bottom" />
-			<child link="UR10_r/base_ideal" />
-			<origin xyz="0.0 0.0 0.555" rpy="0 0 0" />
-		</joint>
+			</joint>
+		</xacro:if>
 	</xacro:unless>
 	<!-- Because one arm is mounted backwards. TODO: use calibrated pose -->
