Commit message: Add support for simplified visuals and update RViz configuration
- Introduced 'use_simple_visuals' launch argument to replace heavy MiR visual meshes with primitives for better RViz/GPU diagnosis.
- Updated multi_mur_base.launch.py, mur620.launch.py, and mur_base.launch.py to include the new argument.
- Enhanced RViz configuration in multi_mur_base.rviz with additional panels, tools, and improved visualization settings for better usability and diagnostics.

File: mir_robot/mir_description/urdf/general/sick_s300.urdf.xacro (robot description, xacro)
@@ -6,14 +6,25 @@
 	<xacro:property name="laser_z" value="0.185" />
 	<xacro:property name="laser_mass" value="2.0" />
-	<xacro:macro name="sick_s300" params="link topic use_simple_collisions:=false">
+	<xacro:macro name="sick_s300" params="link topic use_simple_collisions:=false use_simple_visuals:=false">
 		<link name="${link}">
-			<visual>
-				<origin xyz="0.0 0.0 0.0" rpy="${pi} 0 0" />
-				<geometry>
-					<mesh filename="package://mir_description/meshes/visual/sick_lms-100.stl" />
-				</geometry>
-				<!-- <xacro:insert_block name="material_yellow" /> -->
-				<xacro:insert_block name="material_black" />
-			</visual>
+			<xacro:if value="${use_simple_visuals}">
+				<visual>
+					<origin xyz="0.0 0.0 0.0" rpy="0 0 0" />
+					<geometry>
+						<box size="${laser_x} ${laser_y} ${laser_z}"/>
+					</geometry>
+					<xacro:insert_block name="material_black" />
+				</visual>
+			</xacro:if>
+			<xacro:unless value="${use_simple_visuals}">
+				<visual>
+					<origin xyz="0.0 0.0 0.0" rpy="${pi} 0 0" />
+					<geometry>
+						<mesh filename="package://mir_description/meshes/visual/sick_lms-100.stl" />
+					</geometry>
+					<!-- <xacro:insert_block name="material_yellow" /> -->
+					<xacro:insert_block name="material_black" />
+				</visual>
+			</xacro:unless>
 			<xacro:if value="${use_simple_collisions}">
 				<collision>

File: mir_robot/mir_description/urdf/mir_600/mir_600.urdf.xacro (robot description, xacro)
@@ -29,5 +29,5 @@
 	<xacro:property name="mir_600_match_logo_dy" value="0.330" />
 	<xacro:property name="mir_600_match_logo_dz" value="0.27" />
-	<xacro:macro name="mir_600" params="use_camera:=true use_simple_collisions:=false">
+	<xacro:macro name="mir_600" params="use_camera:=true use_simple_collisions:=false use_simple_visuals:=false">
 		<link name="base_footprint" />
 		<joint name="base_joint" type="fixed">
@@ -40,11 +40,22 @@
 				<origin xyz="${mir_600_act_wheel_dx} 0 0.20" rpy="0 0 0" />
 			</xacro:box_inertial>
-			<visual>
-				<origin xyz="${mir_600_act_wheel_dx} 0 0" rpy="${pi * 0.5} 0 ${pi * 0.5}" />
-				<geometry>
-					<mesh filename="package://mir_description/meshes/visual/mir_600_base.stl"/>
-				</geometry>
-				<xacro:insert_block name="material_white" />
-			</visual>
+			<xacro:if value="${use_simple_visuals}">
+				<visual>
+					<origin xyz="${mir_600_act_wheel_dx} 0 0.20" rpy="0 0 0" />
+					<geometry>
+						<box size="0.9 0.58 0.3"/>
+					</geometry>
+					<xacro:insert_block name="material_white" />
+				</visual>
+			</xacro:if>
+			<xacro:unless value="${use_simple_visuals}">
+				<visual>
+					<origin xyz="${mir_600_act_wheel_dx} 0 0" rpy="${pi * 0.5} 0 ${pi * 0.5}" />
+					<geometry>
+						<mesh filename="package://mir_description/meshes/visual/mir_600_base.stl"/>
+					</geometry>
+					<xacro:insert_block name="material_white" />
+				</visual>
+			</xacro:unless>
 			<xacro:if value="${use_simple_collisions}">
 				<collision>
@@ -86,5 +97,5 @@
 			<origin xyz="0.58985 0.370 0.1914" rpy="0.0 0.0 ${0.25 * pi}" />  <!-- from visually matching up the meshes of the MiR and the laser scanner -->
 		</joint>
-		<xacro:sick_s300 link="front_laser_link" topic="f_scan" use_simple_collisions="${use_simple_collisions}" />
+		<xacro:sick_s300 link="front_laser_link" topic="f_scan" use_simple_collisions="${use_simple_collisions}" use_simple_visuals="${use_simple_visuals}" />
 		<joint name="base_link_to_back_laser_joint" type="fixed">
 			<parent link="base_link" />
@@ -92,5 +103,5 @@
 			<origin xyz="-0.58985 -0.370 0.1914" rpy="0.0 0.0 ${-0.75 * pi}" />  <!-- from visually matching up the meshes of the MiR and the laser scanner -->
 		</joint>
-		<xacro:sick_s300 link="back_laser_link" topic="b_scan" use_simple_collisions="${use_simple_collisions}" />
+		<xacro:sick_s300 link="back_laser_link" topic="b_scan" use_simple_collisions="${use_simple_collisions}" use_simple_visuals="${use_simple_visuals}" />
 		<!-- Ultrasound sensors -->
 		<joint name="us_1_joint" type="fixed">   <!-- right ultrasound -->
@@ -107,10 +118,10 @@
 		<link name="us_2_frame" />
 		<!-- wheels -->
-		<xacro:actuated_wheel locationprefix="left" locationright="-1"/>
-		<xacro:actuated_wheel locationprefix="right" locationright="1"/>
-		<xacro:caster_wheel locationprefix="fl" locationright="-1" wheel_base_dx="${mir_600_front_caster_wheel_base_dx}" use_simple_collisions="${use_simple_collisions}"/>
-		<xacro:caster_wheel locationprefix="fr" locationright="1" wheel_base_dx="${mir_600_front_caster_wheel_base_dx}" use_simple_collisions="${use_simple_collisions}"/>
-		<xacro:caster_wheel locationprefix="bl" locationright="-1" wheel_base_dx="${mir_600_back_caster_wheel_base_dx}" use_simple_collisions="${use_simple_collisions}"/>
-		<xacro:caster_wheel locationprefix="br" locationright="1" wheel_base_dx="${mir_600_back_caster_wheel_base_dx}" use_simple_collisions="${use_simple_collisions}"/>
+		<xacro:actuated_wheel locationprefix="left" locationright="-1" use_simple_visuals="${use_simple_visuals}"/>
+		<xacro:actuated_wheel locationprefix="right" locationright="1" use_simple_visuals="${use_simple_visuals}"/>
+		<xacro:caster_wheel locationprefix="fl" locationright="-1" wheel_base_dx="${mir_600_front_caster_wheel_base_dx}" use_simple_collisions="${use_simple_collisions}" use_simple_visuals="${use_simple_visuals}"/>
+		<xacro:caster_wheel locationprefix="fr" locationright="1" wheel_base_dx="${mir_600_front_caster_wheel_base_dx}" use_simple_collisions="${use_simple_collisions}" use_simple_visuals="${use_simple_visuals}"/>
+		<xacro:caster_wheel locationprefix="bl" locationright="-1" wheel_base_dx="${mir_600_back_caster_wheel_base_dx}" use_simple_collisions="${use_simple_collisions}" use_simple_visuals="${use_simple_visuals}"/>
+		<xacro:caster_wheel locationprefix="br" locationright="1" wheel_base_dx="${mir_600_back_caster_wheel_base_dx}" use_simple_collisions="${use_simple_collisions}" use_simple_visuals="${use_simple_visuals}"/>
 		<joint name="base_link_surface_joint" type="fixed">
 			<origin xyz="${mir_600_act_wheel_dx} 0 0.352" rpy="0 0 0" />
@@ -129,5 +140,5 @@
 		<!-- <xacro:match_logo parent="base_link" locationprefix="left" location_dx="${mir_600_match_logo_dx}" location_dy="${mir_600_match_logo_dy}" location_dz="${mir_600_match_logo_dz}"/>
 		<xacro:match_logo parent="base_link" locationprefix="right" location_dx="${mir_600_match_logo_dx}" location_dy="${-1 * mir_600_match_logo_dy}" location_dz="${mir_600_match_logo_dz}" orientation="${pi}"/> -->
-		<xacro:top_module use_simple_collisions="${use_simple_collisions}"/>
+		<xacro:top_module use_simple_collisions="${use_simple_collisions}" use_simple_visuals="${use_simple_visuals}"/>
 		<!-- Camera -->
 		<!--link name="camera_link">

File: mir_robot/mir_description/urdf/mir_600/mir_600_top_lift.urdf.xacro (robot description, xacro)
@@ -1,16 +1,27 @@
 <?xml version="1.0"?>
 <robot xmlns:xacro="http://ros.org/wiki/xacro">
-    <xacro:macro name="top_lift" params="use_simple_collisions:=false">
+    <xacro:macro name="top_lift" params="use_simple_collisions:=false use_simple_visuals:=false">
         <link name="left_lift_top">
 			<xacro:box_inertial mass="1.0" x="0.2" y="0.2" z="0.3">
 				<origin xyz="0 0 0.15" rpy="0 0 0" />
 			</xacro:box_inertial>
-			<visual>
-				<origin xyz="0 0 0" rpy="${pi * 0.5} 0 ${pi * 0.0}" />
-				<geometry>
-					<mesh filename="package://mir_description/meshes/visual/mir_600_lift_top.stl"/>
-				</geometry>
-				<xacro:insert_block name="material_white" />
-			</visual>
+			<xacro:if value="${use_simple_visuals}">
+				<visual>
+					<origin xyz="0 0 0.15" rpy="0 0 0" />
+					<geometry>
+						<box size="0.2 0.2 0.3"/>
+					</geometry>
+					<xacro:insert_block name="material_white" />
+				</visual>
+			</xacro:if>
+			<xacro:unless value="${use_simple_visuals}">
+				<visual>
+					<origin xyz="0 0 0" rpy="${pi * 0.5} 0 ${pi * 0.0}" />
+					<geometry>
+						<mesh filename="package://mir_description/meshes/visual/mir_600_lift_top.stl"/>
+					</geometry>
+					<xacro:insert_block name="material_white" />
+				</visual>
+			</xacro:unless>
 			<xacro:if value="${use_simple_collisions}">
 				<collision>
@@ -50,11 +61,22 @@
 				<origin xyz="0 0 0.15" rpy="0 0 0" />
 			</xacro:box_inertial>
-			<visual>
-				<origin xyz="0 0 0" rpy="${pi * 0.5} 0 ${pi * 0.0}" />
-				<geometry>
-					<mesh filename="package://mir_description/meshes/visual/mir_600_lift_top.stl"/>
-				</geometry>
-				<xacro:insert_block name="material_white" />
-			</visual>
+			<xacro:if value="${use_simple_visuals}">
+				<visual>
+					<origin xyz="0 0 0.15" rpy="0 0 0" />
+					<geometry>
+						<box size="0.2 0.2 0.3"/>
+					</geometry>
+					<xacro:insert_block name="material_white" />
+				</visual>
+			</xacro:if>
+			<xacro:unless value="${use_simple_visuals}">
+				<visual>
+					<origin xyz="0 0 0" rpy="${pi * 0.5} 0 ${pi * 0.0}" />
+					<geometry>
+						<mesh filename="package://mir_description/meshes/visual/mir_600_lift_top.stl"/>
+					</geometry>
+					<xacro:insert_block name="material_white" />
+				</visual>
+			</xacro:unless>
 			<xacro:if value="${use_simple_collisions}">
 				<collision>

File: mir_robot/mir_description/urdf/mir_600/mir_600_top_module.urdf.xacro (robot description, xacro)
@@ -2,5 +2,5 @@
 <robot xmlns:xacro="http://ros.org/wiki/xacro">
 	<xacro:include filename="$(find mir_description)/urdf/general/common_properties.urdf.xacro" />
-	<xacro:macro name="top_module" params="use_simple_collisions:=false">
+	<xacro:macro name="top_module" params="use_simple_collisions:=false use_simple_visuals:=false">
 		<!-- top module -->
 		<link name="top_module">
@@ -8,11 +8,22 @@
 				<origin xyz="${mir_600_act_wheel_dx} 0 0.25" rpy="0 0 0" />
 			</xacro:box_inertial>
-			<visual>
-				<origin xyz="${mir_600_act_wheel_dx} 0 0" rpy="0 0 ${-pi * 0.5}" />
-				<geometry>
-					<mesh filename="package://mir_description/meshes/visual/mir_600_top_module.stl" scale="0.001 0.001 0.001"/>
-				</geometry>
-				<xacro:insert_block name="material_white" />
-			</visual>
+			<xacro:if value="${use_simple_visuals}">
+				<visual>
+					<origin xyz="${mir_600_act_wheel_dx} 0 0.25" rpy="0 0 0" />
+					<geometry>
+						<box size="1.35 0.91 0.5"/>
+					</geometry>
+					<xacro:insert_block name="material_white" />
+				</visual>
+			</xacro:if>
+			<xacro:unless value="${use_simple_visuals}">
+				<visual>
+					<origin xyz="${mir_600_act_wheel_dx} 0 0" rpy="0 0 ${-pi * 0.5}" />
+					<geometry>
+						<mesh filename="package://mir_description/meshes/visual/mir_600_top_module.stl" scale="0.001 0.001 0.001"/>
+					</geometry>
+					<xacro:insert_block name="material_white" />
+				</visual>
+			</xacro:unless>
 			<collision>
 				<origin xyz="${mir_600_act_wheel_dx} 0 0" rpy="0 0 ${-pi * 0.5}" />
@@ -40,11 +51,22 @@
 				<origin xyz="0 0 0.15" rpy="0 0 0" />
 			</xacro:box_inertial>
-			<visual>
-				<origin xyz="0 0 0" rpy="${pi * 0.5} 0 ${pi * 0.0}" />
-				<geometry>
-					<mesh filename="package://mir_description/meshes/visual/mir_600_lift_bot.stl"/>
-				</geometry>
-				<xacro:insert_block name="material_white" />
-			</visual>
+			<xacro:if value="${use_simple_visuals}">
+				<visual>
+					<origin xyz="0 0 0.15" rpy="0 0 0" />
+					<geometry>
+						<box size="0.2 0.2 0.3"/>
+					</geometry>
+					<xacro:insert_block name="material_white" />
+				</visual>
+			</xacro:if>
+			<xacro:unless value="${use_simple_visuals}">
+				<visual>
+					<origin xyz="0 0 0" rpy="${pi * 0.5} 0 ${pi * 0.0}" />
+					<geometry>
+						<mesh filename="package://mir_description/meshes/visual/mir_600_lift_bot.stl"/>
+					</geometry>
+					<xacro:insert_block name="material_white" />
+				</visual>
+			</xacro:unless>
 			<xacro:if value="${use_simple_collisions}">
 				<collision>
@@ -82,11 +104,22 @@
 				<origin xyz="0 0 0.15" rpy="0 0 0" />
 			</xacro:box_inertial>
-			<visual>
-				<origin xyz="0 0 0" rpy="${pi * 0.5} 0 ${pi * 0.0}" />
-				<geometry>
-					<mesh filename="package://mir_description/meshes/visual/mir_600_lift_bot.stl"/>
-				</geometry>
-				<xacro:insert_block name="material_white" />
-			</visual>
+			<xacro:if value="${use_simple_visuals}">
+				<visual>
+					<origin xyz="0 0 0.15" rpy="0 0 0" />
+					<geometry>
+						<box size="0.2 0.2 0.3"/>
+					</geometry>
+					<xacro:insert_block name="material_white" />
+				</visual>
+			</xacro:if>
+			<xacro:unless value="${use_simple_visuals}">
+				<visual>
+					<origin xyz="0 0 0" rpy="${pi * 0.5} 0 ${pi * 0.0}" />
+					<geometry>
+						<mesh filename="package://mir_description/meshes/visual/mir_600_lift_bot.stl"/>
+					</geometry>
+					<xacro:insert_block name="material_white" />
+				</visual>
+			</xacro:unless>
 			<xacro:if value="${use_simple_collisions}">
 				<collision>

File: mir_robot/mir_description/urdf/mir_600/mir_600_wheels.urdf.xacro (robot description, xacro)
@@ -2,5 +2,5 @@
 <robot xmlns:xacro="http://ros.org/wiki/xacro">
 	<xacro:include filename="$(find mir_description)/urdf/general/common_properties.urdf.xacro" />
-	<xacro:macro name="actuated_wheel" params="locationprefix locationright">
+	<xacro:macro name="actuated_wheel" params="locationprefix locationright use_simple_visuals:=false">
 		<joint name="${locationprefix}_wheel_joint" type="continuous">
 			<origin xyz="0.0 ${-mir_600_act_wheel_dy * locationright} ${mir_600_act_wheel_radius}" rpy="0 0 0" />
@@ -14,11 +14,22 @@
 				<origin xyz="0 0 0" rpy="${0.5 * pi} 0 0" />
 			</xacro:cylinder_inertial>
-			<visual>
-				<origin xyz="0 ${locationright * mir_600_act_wheel_width*0.5} 0" rpy="${pi * 0.5} 0 ${0.5 * pi * (1+ locationright)}" />
-				<geometry>
-					<mesh filename="package://mir_description/meshes/visual/mir_600_wheel.stl" />
-				</geometry>
-				<xacro:insert_block name="material_dark_grey" />
-			</visual>
+			<xacro:if value="${use_simple_visuals}">
+				<visual>
+					<origin xyz="0 0 0" rpy="${pi * 0.5} 0 ${pi * -1}" />
+					<geometry>
+						<cylinder radius="${mir_600_act_wheel_radius}" length="${mir_600_act_wheel_width}"/>
+					</geometry>
+					<xacro:insert_block name="material_dark_grey" />
+				</visual>
+			</xacro:if>
+			<xacro:unless value="${use_simple_visuals}">
+				<visual>
+					<origin xyz="0 ${locationright * mir_600_act_wheel_width*0.5} 0" rpy="${pi * 0.5} 0 ${0.5 * pi * (1+ locationright)}" />
+					<geometry>
+						<mesh filename="package://mir_description/meshes/visual/mir_600_wheel.stl" />
+					</geometry>
+					<xacro:insert_block name="material_dark_grey" />
+				</visual>
+			</xacro:unless>
 			<collision>
 				<origin xyz="0 0 0" rpy="${pi * 0.5} 0 ${pi * -1}" />
@@ -29,5 +40,5 @@
 		</link>
 	</xacro:macro>
-	<xacro:macro name="caster_wheel" params="locationprefix locationright wheel_base_dx use_simple_collisions:=false">
+	<xacro:macro name="caster_wheel" params="locationprefix locationright wheel_base_dx use_simple_collisions:=false use_simple_visuals:=false">
 		<!-- caster hub -->
 		<joint name="${locationprefix}_caster_rotation_joint" type="continuous">
@@ -51,11 +62,22 @@
 				izz="0.00017923555074" />
 		</inertial>
-		<visual>
-			<origin xyz="0 0 0" rpy="0 0 0" />
-			<geometry>
-				<mesh filename="package://mir_description/meshes/visual/caster_wheel_base.stl" />
-			</geometry>
-			<xacro:insert_block name="material_silver" />
-		</visual>
+		<xacro:if value="${use_simple_visuals}">
+			<visual>
+				<origin xyz="0 0 -0.03" rpy="0 0 0" />
+				<geometry>
+					<box size="0.16 0.12 0.08"/>
+				</geometry>
+				<xacro:insert_block name="material_silver" />
+			</visual>
+		</xacro:if>
+		<xacro:unless value="${use_simple_visuals}">
+			<visual>
+				<origin xyz="0 0 0" rpy="0 0 0" />
+				<geometry>
+					<mesh filename="package://mir_description/meshes/visual/caster_wheel_base.stl" />
+				</geometry>
+				<xacro:insert_block name="material_silver" />
+			</visual>
+		</xacro:unless>
 		<xacro:if value="${use_simple_collisions}">
 			<collision>
@@ -86,11 +108,22 @@
 				<origin xyz="0 0 0" rpy="${0.5 * pi} 0 0" />
 			</xacro:cylinder_inertial>
-			<visual>
-				<origin xyz="0 0 0" rpy="${pi * 0.5} 0 0" />
-				<geometry>
-					<mesh filename="package://mir_description/meshes/visual/mir_600_caster_wheel.stl" />
-				</geometry>
-				<xacro:insert_block name="material_dark_grey" />
-			</visual>
+			<xacro:if value="${use_simple_visuals}">
+				<visual>
+					<origin xyz="0 0 0" rpy="${pi * 0.5} 0 0" />
+					<geometry>
+						<cylinder radius="${mir_600_caster_wheel_radius}" length="${mir_600_caster_wheel_width}"/>
+					</geometry>
+					<xacro:insert_block name="material_dark_grey" />
+				</visual>
+			</xacro:if>
+			<xacro:unless value="${use_simple_visuals}">
+				<visual>
+					<origin xyz="0 0 0" rpy="${pi * 0.5} 0 0" />
+					<geometry>
+						<mesh filename="package://mir_description/meshes/visual/mir_600_caster_wheel.stl" />
+					</geometry>
+					<xacro:insert_block name="material_dark_grey" />
+				</visual>
+			</xacro:unless>
 			<collision>
 				<origin xyz="0 0 0" rpy="${pi * 0.5} 0 0" />

File: mur_robot/mur_description/urdf/mur_620.gazebo.xacro (robot description, xacro)
@@ -11,4 +11,6 @@
 	<xacro:arg name="use_simple_collisions" default='false'/>
 	<xacro:property name="use_simple_collisions" value="$(arg use_simple_collisions)"/>
+	<xacro:arg name="use_simple_visuals" default='false'/>
+	<xacro:property name="use_simple_visuals" value="$(arg use_simple_visuals)"/>
 	<xacro:arg name="use_lift" default='true'/>
 	<xacro:property name="use_lift" value="$(arg use_lift)"/>
@@ -47,4 +49,5 @@
 		use_camera="$(arg use_camera)"
 		use_simple_collisions="$(arg use_simple_collisions)"
+		use_simple_visuals="$(arg use_simple_visuals)"
 	/>
 	<!-- Init the MiR600 macro that includes all infos that Gazebo need to function -->
@@ -107,5 +110,5 @@
 	<!-- Init the lift macro -->
 	<xacro:if value="${use_lift}">
-		<xacro:top_lift use_simple_collisions="$(arg use_simple_collisions)"/>
+		<xacro:top_lift use_simple_collisions="$(arg use_simple_collisions)" use_simple_visuals="$(arg use_simple_visuals)"/>
 		<xacro:if value="${use_arms}">
 			<joint name="plattform_manipulator_joint_l" type="fixed">
