Commit message: Enhance visual mesh options and improve RViz configuration
- Updated URDF macros for wheels and casters to include new parameters for high-quality visual meshes.
- Added launch arguments for high-quality visuals and specific visual mesh options in multi_mur620.launch.py, multi_mur_base.launch.py, mur620.launch.py, and mur_base.launch.py.
- Modified gazebo.xacro to utilize new visual mesh parameters for lift and caster components.
- Enhanced RViz configuration with improved panel sizes and view settings for better usability.
- Removed redundant visual settings for UR10 robot links in RViz configuration to streamline the display.

File: mir_robot/mir_description/urdf/general/sick_s300.urdf.xacro (robot description, xacro)
@@ -6,7 +6,7 @@
 	<xacro:property name="laser_z" value="0.185" />
 	<xacro:property name="laser_mass" value="2.0" />
-	<xacro:macro name="sick_s300" params="link topic use_simple_collisions:=false use_simple_visuals:=false">
+	<xacro:macro name="sick_s300" params="link topic use_simple_collisions:=false use_simple_visuals:=false use_laser_visual_mesh:=false">
 		<link name="${link}">
-			<xacro:if value="${use_simple_visuals}">
+			<xacro:if value="${use_simple_visuals and not use_laser_visual_mesh}">
 				<visual>
 					<origin xyz="0.0 0.0 0.0" rpy="0 0 0" />
@@ -17,5 +17,5 @@
 				</visual>
 			</xacro:if>
-			<xacro:unless value="${use_simple_visuals}">
+			<xacro:unless value="${use_simple_visuals and not use_laser_visual_mesh}">
 				<visual>
 					<origin xyz="0.0 0.0 0.0" rpy="${pi} 0 0" />

File: mir_robot/mir_description/urdf/mir_600/mir_600.urdf.xacro (robot description, xacro)
@@ -29,5 +29,5 @@
 	<xacro:property name="mir_600_match_logo_dy" value="0.330" />
 	<xacro:property name="mir_600_match_logo_dz" value="0.27" />
-	<xacro:macro name="mir_600" params="use_camera:=true use_simple_collisions:=false use_simple_visuals:=false">
+	<xacro:macro name="mir_600" params="use_camera:=true use_simple_collisions:=false use_simple_visuals:=false use_high_quality_visuals:=false use_base_visual_mesh:=false use_top_visual_mesh:=false use_wheel_visual_mesh:=false use_caster_visual_mesh:=false use_lift_visual_mesh:=false use_laser_visual_mesh:=false">
 		<link name="base_footprint" />
 		<joint name="base_joint" type="fixed">
@@ -40,5 +40,5 @@
 				<origin xyz="${mir_600_act_wheel_dx} 0 0.20" rpy="0 0 0" />
 			</xacro:box_inertial>
-			<xacro:if value="${use_simple_visuals}">
+			<xacro:if value="${use_simple_visuals and not use_base_visual_mesh}">
 				<visual>
 					<origin xyz="${mir_600_act_wheel_dx} 0 0.20" rpy="0 0 0" />
@@ -49,9 +49,14 @@
 				</visual>
 			</xacro:if>
-			<xacro:unless value="${use_simple_visuals}">
+			<xacro:unless value="${use_simple_visuals and not use_base_visual_mesh}">
 				<visual>
 					<origin xyz="${mir_600_act_wheel_dx} 0 0" rpy="${pi * 0.5} 0 ${pi * 0.5}" />
 					<geometry>
-						<mesh filename="package://mir_description/meshes/visual/mir_600_base.stl"/>
+						<xacro:if value="${use_high_quality_visuals}">
+							<mesh filename="package://mir_description/meshes/visual/mir_600_base.stl"/>
+						</xacro:if>
+						<xacro:unless value="${use_high_quality_visuals}">
+							<mesh filename="package://mir_description/meshes/visual/simplify_mir_600_base.stl"/>
+						</xacro:unless>
 					</geometry>
 					<xacro:insert_block name="material_white" />
@@ -97,5 +102,5 @@
 			<origin xyz="0.58985 0.370 0.1914" rpy="0.0 0.0 ${0.25 * pi}" />  <!-- from visually matching up the meshes of the MiR and the laser scanner -->
 		</joint>
-		<xacro:sick_s300 link="front_laser_link" topic="f_scan" use_simple_collisions="${use_simple_collisions}" use_simple_visuals="${use_simple_visuals}" />
+		<xacro:sick_s300 link="front_laser_link" topic="f_scan" use_simple_collisions="${use_simple_collisions}" use_simple_visuals="${use_simple_visuals}" use_laser_visual_mesh="${use_laser_visual_mesh}" />
 		<joint name="base_link_to_back_laser_joint" type="fixed">
 			<parent link="base_link" />
@@ -103,5 +108,5 @@
 			<origin xyz="-0.58985 -0.370 0.1914" rpy="0.0 0.0 ${-0.75 * pi}" />  <!-- from visually matching up the meshes of the MiR and the laser scanner -->
 		</joint>
-		<xacro:sick_s300 link="back_laser_link" topic="b_scan" use_simple_collisions="${use_simple_collisions}" use_simple_visuals="${use_simple_visuals}" />
+		<xacro:sick_s300 link="back_laser_link" topic="b_scan" use_simple_collisions="${use_simple_collisions}" use_simple_visuals="${use_simple_visuals}" use_laser_visual_mesh="${use_laser_visual_mesh}" />
 		<!-- Ultrasound sensors -->
 		<joint name="us_1_joint" type="fixed">   <!-- right ultrasound -->
@@ -118,10 +123,10 @@
 		<link name="us_2_frame" />
 		<!-- wheels -->
-		<xacro:actuated_wheel locationprefix="left" locationright="-1" use_simple_visuals="${use_simple_visuals}"/>
-		<xacro:actuated_wheel locationprefix="right" locationright="1" use_simple_visuals="${use_simple_visuals}"/>
-		<xacro:caster_wheel locationprefix="fl" locationright="-1" wheel_base_dx="${mir_600_front_caster_wheel_base_dx}" use_simple_collisions="${use_simple_collisions}" use_simple_visuals="${use_simple_visuals}"/>
-		<xacro:caster_wheel locationprefix="fr" locationright="1" wheel_base_dx="${mir_600_front_caster_wheel_base_dx}" use_simple_collisions="${use_simple_collisions}" use_simple_visuals="${use_simple_visuals}"/>
-		<xacro:caster_wheel locationprefix="bl" locationright="-1" wheel_base_dx="${mir_600_back_caster_wheel_base_dx}" use_simple_collisions="${use_simple_collisions}" use_simple_visuals="${use_simple_visuals}"/>
-		<xacro:caster_wheel locationprefix="br" locationright="1" wheel_base_dx="${mir_600_back_caster_wheel_base_dx}" use_simple_collisions="${use_simple_collisions}" use_simple_visuals="${use_simple_visuals}"/>
+		<xacro:actuated_wheel locationprefix="left" locationright="-1" use_simple_visuals="${use_simple_visuals}" use_wheel_visual_mesh="${use_wheel_visual_mesh}"/>
+		<xacro:actuated_wheel locationprefix="right" locationright="1" use_simple_visuals="${use_simple_visuals}" use_wheel_visual_mesh="${use_wheel_visual_mesh}"/>
+		<xacro:caster_wheel locationprefix="fl" locationright="-1" wheel_base_dx="${mir_600_front_caster_wheel_base_dx}" use_simple_collisions="${use_simple_collisions}" use_simple_visuals="${use_simple_visuals}" use_caster_visual_mesh="${use_caster_visual_mesh}"/>
+		<xacro:caster_wheel locationprefix="fr" locationright="1" wheel_base_dx="${mir_600_front_caster_wheel_base_dx}" use_simple_collisions="${use_simple_collisions}" use_simple_visuals="${use_simple_visuals}" use_caster_visual_mesh="${use_caster_visual_mesh}"/>
+		<xacro:caster_wheel locationprefix="bl" locationright="-1" wheel_base_dx="${mir_600_back_caster_wheel_base_dx}" use_simple_collisions="${use_simple_collisions}" use_simple_visuals="${use_simple_visuals}" use_caster_visual_mesh="${use_caster_visual_mesh}"/>
+		<xacro:caster_wheel locationprefix="br" locationright="1" wheel_base_dx="${mir_600_back_caster_wheel_base_dx}" use_simple_collisions="${use_simple_collisions}" use_simple_visuals="${use_simple_visuals}" use_caster_visual_mesh="${use_caster_visual_mesh}"/>
 		<joint name="base_link_surface_joint" type="fixed">
 			<origin xyz="${mir_600_act_wheel_dx} 0 0.352" rpy="0 0 0" />
@@ -140,5 +145,5 @@
 		<!-- <xacro:match_logo parent="base_link" locationprefix="left" location_dx="${mir_600_match_logo_dx}" location_dy="${mir_600_match_logo_dy}" location_dz="${mir_600_match_logo_dz}"/>
 		<xacro:match_logo parent="base_link" locationprefix="right" location_dx="${mir_600_match_logo_dx}" location_dy="${-1 * mir_600_match_logo_dy}" location_dz="${mir_600_match_logo_dz}" orientation="${pi}"/> -->
-		<xacro:top_module use_simple_collisions="${use_simple_collisions}" use_simple_visuals="${use_simple_visuals}"/>
+		<xacro:top_module use_simple_collisions="${use_simple_collisions}" use_simple_visuals="${use_simple_visuals}" use_high_quality_visuals="${use_high_quality_visuals}" use_top_visual_mesh="${use_top_visual_mesh}" use_lift_visual_mesh="${use_lift_visual_mesh}"/>
 		<!-- Camera -->
 		<!--link name="camera_link">

File: mir_robot/mir_description/urdf/mir_600/mir_600_top_lift.urdf.xacro (robot description, xacro)
@@ -1,10 +1,10 @@
 <?xml version="1.0"?>
 <robot xmlns:xacro="http://ros.org/wiki/xacro">
-    <xacro:macro name="top_lift" params="use_simple_collisions:=false use_simple_visuals:=false">
+    <xacro:macro name="top_lift" params="use_simple_collisions:=false use_simple_visuals:=false use_lift_visual_mesh:=false">
         <link name="left_lift_top">
 			<xacro:box_inertial mass="1.0" x="0.2" y="0.2" z="0.3">
 				<origin xyz="0 0 0.15" rpy="0 0 0" />
 			</xacro:box_inertial>
-			<xacro:if value="${use_simple_visuals}">
+			<xacro:if value="${use_simple_visuals and not use_lift_visual_mesh}">
 				<visual>
 					<origin xyz="0 0 0.15" rpy="0 0 0" />
@@ -15,5 +15,5 @@
 				</visual>
 			</xacro:if>
-			<xacro:unless value="${use_simple_visuals}">
+			<xacro:unless value="${use_simple_visuals and not use_lift_visual_mesh}">
 				<visual>
 					<origin xyz="0 0 0" rpy="${pi * 0.5} 0 ${pi * 0.0}" />
@@ -61,5 +61,5 @@
 				<origin xyz="0 0 0.15" rpy="0 0 0" />
 			</xacro:box_inertial>
-			<xacro:if value="${use_simple_visuals}">
+			<xacro:if value="${use_simple_visuals and not use_lift_visual_mesh}">
 				<visual>
 					<origin xyz="0 0 0.15" rpy="0 0 0" />
@@ -70,5 +70,5 @@
 				</visual>
 			</xacro:if>
-			<xacro:unless value="${use_simple_visuals}">
+			<xacro:unless value="${use_simple_visuals and not use_lift_visual_mesh}">
 				<visual>
 					<origin xyz="0 0 0" rpy="${pi * 0.5} 0 ${pi * 0.0}" />

File: mir_robot/mir_description/urdf/mir_600/mir_600_top_module.urdf.xacro (robot description, xacro)
@@ -2,5 +2,5 @@
 <robot xmlns:xacro="http://ros.org/wiki/xacro">
 	<xacro:include filename="$(find mir_description)/urdf/general/common_properties.urdf.xacro" />
-	<xacro:macro name="top_module" params="use_simple_collisions:=false use_simple_visuals:=false">
+	<xacro:macro name="top_module" params="use_simple_collisions:=false use_simple_visuals:=false use_high_quality_visuals:=false use_top_visual_mesh:=false use_lift_visual_mesh:=false">
 		<!-- top module -->
 		<link name="top_module">
@@ -8,5 +8,5 @@
 				<origin xyz="${mir_600_act_wheel_dx} 0 0.25" rpy="0 0 0" />
 			</xacro:box_inertial>
-			<xacro:if value="${use_simple_visuals}">
+			<xacro:if value="${use_simple_visuals and not use_top_visual_mesh}">
 				<visual>
 					<origin xyz="${mir_600_act_wheel_dx} 0 0.25" rpy="0 0 0" />
@@ -17,19 +17,34 @@
 				</visual>
 			</xacro:if>
-			<xacro:unless value="${use_simple_visuals}">
+			<xacro:unless value="${use_simple_visuals and not use_top_visual_mesh}">
 				<visual>
 					<origin xyz="${mir_600_act_wheel_dx} 0 0" rpy="0 0 ${-pi * 0.5}" />
 					<geometry>
-						<mesh filename="package://mir_description/meshes/visual/mir_600_top_module.stl" scale="0.001 0.001 0.001"/>
+						<xacro:if value="${use_high_quality_visuals}">
+							<mesh filename="package://mir_description/meshes/visual/mir_600_top_module.stl" scale="0.001 0.001 0.001"/>
+						</xacro:if>
+						<xacro:unless value="${use_high_quality_visuals}">
+							<mesh filename="package://mir_description/meshes/visual/simplify_mir_600_top_module.stl" scale="0.001 0.001 0.001"/>
+						</xacro:unless>
 					</geometry>
 					<xacro:insert_block name="material_white" />
 				</visual>
 			</xacro:unless>
-			<collision>
-				<origin xyz="${mir_600_act_wheel_dx} 0 0" rpy="0 0 ${-pi * 0.5}" />
-				<geometry>
-					<mesh filename="package://mir_description/meshes/collision/mir_600_top_module.stl" scale="0.001 0.001 0.001" />
-				</geometry>
-			</collision>
+			<xacro:if value="${use_simple_collisions}">
+				<collision>
+					<origin xyz="${mir_600_act_wheel_dx} 0 0.25" rpy="0 0 0" />
+					<geometry>
+						<box size="1.35 0.91 0.5"/>
+					</geometry>
+				</collision>
+			</xacro:if>
+			<xacro:unless value="${use_simple_collisions}">
+				<collision>
+					<origin xyz="${mir_600_act_wheel_dx} 0 0" rpy="0 0 ${-pi * 0.5}" />
+					<geometry>
+						<mesh filename="package://mir_description/meshes/collision/mir_600_top_module.stl" scale="0.001 0.001 0.001" />
+					</geometry>
+				</collision>
+			</xacro:unless>
 		</link>
 		<gazebo reference="top_module">
@@ -51,5 +66,5 @@
 				<origin xyz="0 0 0.15" rpy="0 0 0" />
 			</xacro:box_inertial>
-			<xacro:if value="${use_simple_visuals}">
+			<xacro:if value="${use_simple_visuals and not use_lift_visual_mesh}">
 				<visual>
 					<origin xyz="0 0 0.15" rpy="0 0 0" />
@@ -60,5 +75,5 @@
 				</visual>
 			</xacro:if>
-			<xacro:unless value="${use_simple_visuals}">
+			<xacro:unless value="${use_simple_visuals and not use_lift_visual_mesh}">
 				<visual>
 					<origin xyz="0 0 0" rpy="${pi * 0.5} 0 ${pi * 0.0}" />
@@ -104,5 +119,5 @@
 				<origin xyz="0 0 0.15" rpy="0 0 0" />
 			</xacro:box_inertial>
-			<xacro:if value="${use_simple_visuals}">
+			<xacro:if value="${use_simple_visuals and not use_lift_visual_mesh}">
 				<visual>
 					<origin xyz="0 0 0.15" rpy="0 0 0" />
@@ -113,5 +128,5 @@
 				</visual>
 			</xacro:if>
-			<xacro:unless value="${use_simple_visuals}">
+			<xacro:unless value="${use_simple_visuals and not use_lift_visual_mesh}">
 				<visual>
 					<origin xyz="0 0 0" rpy="${pi * 0.5} 0 ${pi * 0.0}" />

File: mir_robot/mir_description/urdf/mir_600/mir_600_wheels.urdf.xacro (robot description, xacro)
@@ -2,5 +2,5 @@
 <robot xmlns:xacro="http://ros.org/wiki/xacro">
 	<xacro:include filename="$(find mir_description)/urdf/general/common_properties.urdf.xacro" />
-	<xacro:macro name="actuated_wheel" params="locationprefix locationright use_simple_visuals:=false">
+	<xacro:macro name="actuated_wheel" params="locationprefix locationright use_simple_visuals:=false use_wheel_visual_mesh:=false">
 		<joint name="${locationprefix}_wheel_joint" type="continuous">
 			<origin xyz="0.0 ${-mir_600_act_wheel_dy * locationright} ${mir_600_act_wheel_radius}" rpy="0 0 0" />
@@ -14,5 +14,5 @@
 				<origin xyz="0 0 0" rpy="${0.5 * pi} 0 0" />
 			</xacro:cylinder_inertial>
-			<xacro:if value="${use_simple_visuals}">
+			<xacro:if value="${not use_wheel_visual_mesh}">
 				<visual>
 					<origin xyz="0 0 0" rpy="${pi * 0.5} 0 ${pi * -1}" />
@@ -23,5 +23,5 @@
 				</visual>
 			</xacro:if>
-			<xacro:unless value="${use_simple_visuals}">
+			<xacro:unless value="${not use_wheel_visual_mesh}">
 				<visual>
 					<origin xyz="0 ${locationright * mir_600_act_wheel_width*0.5} 0" rpy="${pi * 0.5} 0 ${0.5 * pi * (1+ locationright)}" />
@@ -40,5 +40,5 @@
 		</link>
 	</xacro:macro>
-	<xacro:macro name="caster_wheel" params="locationprefix locationright wheel_base_dx use_simple_collisions:=false use_simple_visuals:=false">
+	<xacro:macro name="caster_wheel" params="locationprefix locationright wheel_base_dx use_simple_collisions:=false use_simple_visuals:=false use_caster_visual_mesh:=false">
 		<!-- caster hub -->
 		<joint name="${locationprefix}_caster_rotation_joint" type="continuous">
@@ -62,5 +62,5 @@
 				izz="0.00017923555074" />
 		</inertial>
-		<xacro:if value="${use_simple_visuals}">
+		<xacro:if value="${use_simple_visuals and not use_caster_visual_mesh}">
 			<visual>
 				<origin xyz="0 0 -0.03" rpy="0 0 0" />
@@ -71,5 +71,5 @@
 			</visual>
 		</xacro:if>
-		<xacro:unless value="${use_simple_visuals}">
+		<xacro:unless value="${use_simple_visuals and not use_caster_visual_mesh}">
 			<visual>
 				<origin xyz="0 0 0" rpy="0 0 0" />
@@ -108,5 +108,5 @@
 				<origin xyz="0 0 0" rpy="${0.5 * pi} 0 0" />
 			</xacro:cylinder_inertial>
-			<xacro:if value="${use_simple_visuals}">
+			<xacro:if value="${use_simple_visuals and not use_caster_visual_mesh}">
 				<visual>
 					<origin xyz="0 0 0" rpy="${pi * 0.5} 0 0" />
@@ -117,5 +117,5 @@
 				</visual>
 			</xacro:if>
-			<xacro:unless value="${use_simple_visuals}">
+			<xacro:unless value="${use_simple_visuals and not use_caster_visual_mesh}">
 				<visual>
 					<origin xyz="0 0 0" rpy="${pi * 0.5} 0 0" />

File: mur_robot/mur_description/urdf/mur_620.gazebo.xacro (robot description, xacro)
@@ -13,4 +13,11 @@
 	<xacro:arg name="use_simple_visuals" default='false'/>
 	<xacro:property name="use_simple_visuals" value="$(arg use_simple_visuals)"/>
+	<xacro:arg name="use_high_quality_visuals" default='false'/>
+	<xacro:arg name="use_base_visual_mesh" default='false'/>
+	<xacro:arg name="use_top_visual_mesh" default='false'/>
+	<xacro:arg name="use_wheel_visual_mesh" default='false'/>
+	<xacro:arg name="use_caster_visual_mesh" default='false'/>
+	<xacro:arg name="use_lift_visual_mesh" default='false'/>
+	<xacro:arg name="use_laser_visual_mesh" default='false'/>
 	<xacro:arg name="use_lift" default='true'/>
 	<xacro:property name="use_lift" value="$(arg use_lift)"/>
@@ -50,4 +57,11 @@
 		use_simple_collisions="$(arg use_simple_collisions)"
 		use_simple_visuals="$(arg use_simple_visuals)"
+		use_high_quality_visuals="$(arg use_high_quality_visuals)"
+		use_base_visual_mesh="$(arg use_base_visual_mesh)"
+		use_top_visual_mesh="$(arg use_top_visual_mesh)"
+		use_wheel_visual_mesh="$(arg use_wheel_visual_mesh)"
+		use_caster_visual_mesh="$(arg use_caster_visual_mesh)"
+		use_lift_visual_mesh="$(arg use_lift_visual_mesh)"
+		use_laser_visual_mesh="$(arg use_laser_visual_mesh)"
 	/>
 	<!-- Init the MiR600 macro that includes all infos that Gazebo need to function -->
@@ -110,5 +124,5 @@
 	<!-- Init the lift macro -->
 	<xacro:if value="${use_lift}">
-		<xacro:top_lift use_simple_collisions="$(arg use_simple_collisions)" use_simple_visuals="$(arg use_simple_visuals)"/>
+		<xacro:top_lift use_simple_collisions="$(arg use_simple_collisions)" use_simple_visuals="$(arg use_simple_visuals)" use_lift_visual_mesh="$(arg use_lift_visual_mesh)"/>
 		<xacro:if value="${use_arms}">
 			<joint name="plattform_manipulator_joint_l" type="fixed">
