Commit message: lidar wip

File: mir_robot/mir_description/urdf/general/plugins.gazebo.xacro (robot description, xacro)
@@ -12,4 +12,11 @@
 					<legacyModeNS>true</legacyModeNS>
 				</ros>
+			</plugin>
+		</gazebo>
+	</xacro:macro>
+	<xacro:macro name="gazebo_sim_sensors" params="robot_namespace">
+		<gazebo>
+			<plugin filename="gz-sim-sensors-system" name="gz::sim::systems::Sensors">
+				<render_engine>ogre2</render_engine>
 			</plugin>
 		</gazebo>

Commit message: Add new frames and update run script for simulation
- Added new PDF files for frames captured on 2026-05-21 at 13:59:52 and 14:06:30.
- Introduced a new Graphviz file for visualizing the transformation frames.
- Updated the run_mur.sh script to include additional launch parameters: moveit_robot set to 'all' and fake_localization enabled.

File: mir_robot/mir_description/urdf/general/plugins.gazebo.xacro (robot description, xacro)
@@ -13,5 +13,5 @@
 		</gazebo>
 	</xacro:macro>
-	<xacro:macro name="gazebo_sim_sensors" params="robot_namespace">
+	<xacro:macro name="gazebo_sim_sensors" params="robot_namespace use_lidar:=true">
 		<gazebo>
 			<xacro:if value="${robot_namespace == 'mur620a'}">
@@ -22,16 +22,18 @@
 			</xacro:if>
 		</gazebo>
-		<xacro:sick_s300_gazebo
-			link="front_laser_link"
-			topic="${robot_namespace}/f_scan"
-			robot_namespace="${robot_namespace}"
-			tf_prefix=""
-		/>
-		<xacro:sick_s300_gazebo
-			link="back_laser_link"
-			topic="${robot_namespace}/b_scan"
-			robot_namespace="${robot_namespace}"
-			tf_prefix=""
-		/>
+		<xacro:if value="${use_lidar == 'true'}">
+			<xacro:sick_s300_gazebo
+				link="front_laser_link"
+				topic="${robot_namespace}/f_scan"
+				robot_namespace="${robot_namespace}"
+				tf_prefix=""
+			/>
+			<xacro:sick_s300_gazebo
+				link="back_laser_link"
+				topic="${robot_namespace}/b_scan"
+				robot_namespace="${robot_namespace}"
+				tf_prefix=""
+			/>
+		</xacro:if>
 	</xacro:macro>
 	<!-- This controller is deprecated and forbidden in Noetic -->

File: mir_robot/mir_description/urdf/mir_600/mir_600.gazebo.xacro (robot description, xacro)
@@ -8,5 +8,5 @@
 	<xacro:include filename="$(find mir_description)/urdf/general/_d435.gazebo.xacro" />
 	<xacro:property name="imu_standard_deviation" value="0.00017" />
-	<xacro:macro name="mir_600_gazebo" params="tf_prefix robot_namespace use_camera:=true">
+	<xacro:macro name="mir_600_gazebo" params="tf_prefix robot_namespace use_camera:=true use_lidar:=true">
 		<!-- Predefine some values that are necessary later. It is important to differenciate between empty and not empty robot_namespace and tf_prefix -->
 		<xacro:if value="${robot_namespace == ''}">
@@ -46,8 +46,10 @@
 		<!-- Add transmissions to wheels -->
 		<xacro:mir_600_wheel_transmissions/>
-		<!-- Add Gazebo xacro for the laser scanner to work in Gazebo -->
-		<!-- Please match there macro calls with the sick_s300 xacro calls in the mir_600.urdf.xacro file-->
-		<xacro:sick_s300_gazebo link="front_laser_link" robot_namespace="${robot_namespace_slashed}" topic="${tf_prefix_slashed}f_scan" tf_prefix="${tf_prefix_slashed}"/>
-		<xacro:sick_s300_gazebo link="back_laser_link" robot_namespace="${robot_namespace_slashed}" topic="${tf_prefix_slashed}b_scan" tf_prefix="${tf_prefix_slashed}"/>
+		<xacro:if value="${use_lidar == 'true'}">
+			<!-- Add Gazebo xacro for the laser scanner to work in Gazebo -->
+			<!-- Please match there macro calls with the sick_s300 xacro calls in the mir_600.urdf.xacro file-->
+			<xacro:sick_s300_gazebo link="front_laser_link" robot_namespace="${robot_namespace_slashed}" topic="${tf_prefix_slashed}f_scan" tf_prefix="${tf_prefix_slashed}"/>
+			<xacro:sick_s300_gazebo link="back_laser_link" robot_namespace="${robot_namespace_slashed}" topic="${tf_prefix_slashed}b_scan" tf_prefix="${tf_prefix_slashed}"/>
+		</xacro:if>
 		<xacro:if value="${use_camera}">
 			<!-- Settings for the camera of the robot to work in the simulation environment-->

File: mur_robot/mur_description/urdf/mur_620.gazebo.xacro (robot description, xacro)
@@ -20,4 +20,5 @@
 	<xacro:arg name="use_lift_visual_mesh" default='false'/>
 	<xacro:arg name="use_laser_visual_mesh" default='false'/>
+	<xacro:arg name="use_lidar" default='true'/>
 	<xacro:arg name="use_lift" default='true'/>
 	<xacro:property name="use_lift" value="$(arg use_lift)"/>
@@ -66,5 +67,5 @@
 	/>
 	<!-- Init the MiR600 macro that includes all infos that Gazebo need to function -->
-	<xacro:mir_600_gazebo tf_prefix="$(arg tf_prefix_mir)" robot_namespace="$(arg robot_namespace)" use_camera="$(arg use_camera)"/>
+	<xacro:mir_600_gazebo tf_prefix="$(arg tf_prefix_mir)" robot_namespace="$(arg robot_namespace)" use_camera="$(arg use_camera)" use_lidar="$(arg use_lidar)"/>
 	<!-- Init the plugins that run the MiR in Gazebo -->
 	<xacro:controller_plugin_gazebo
@@ -72,5 +73,5 @@
 		controllers_file="$(arg simulation_controllers)"
 	/>
-	<xacro:gazebo_sim_sensors robot_namespace="$(arg robot_namespace)"/>
+	<xacro:gazebo_sim_sensors robot_namespace="$(arg robot_namespace)" use_lidar="$(arg use_lidar)"/>
 	<xacro:mir_robot_ros2_control/>
 	<xacro:if value="${use_arms}">
