Commit message: Fix Jazzy MuR simulation startup and workspace bootstrap

File: mir_robot/mir_description/urdf/general/plugins.gazebo.xacro (robot description, xacro)
@@ -3,5 +3,5 @@
 	<xacro:macro name="controller_plugin_gazebo" params="robot_namespace controllers_file">
 		<gazebo>
-			<plugin filename="libgz_ros2_control-system.so" name="gz_ros2_control::GazeboSimROS2ControlPlugin">
+			<plugin filename="gz_ros2_control-system" name="gz_ros2_control::GazeboSimROS2ControlPlugin">
 				<parameters>${controllers_file}</parameters>
 				<ros>
@@ -13,7 +13,7 @@
 		</gazebo>
 	</xacro:macro>
-	<xacro:macro name="gazebo_sim_sensors" params="robot_namespace use_lidar:=true">
+	<xacro:macro name="gazebo_sim_sensors" params="robot_namespace use_lidar:=true enable_sensors:=true">
 		<gazebo>
-			<xacro:if value="${robot_namespace == 'mur620a'}">
+			<xacro:if value="${robot_namespace == 'mur620a' and enable_sensors == 'true'}">
 				<plugin filename="gz-sim-sensors-system" name="gz::sim::systems::Sensors">
 					<render_engine>ogre2</render_engine>

File: mur_robot/mur_description/urdf/mur_620.gazebo.xacro (robot description, xacro)
@@ -21,4 +21,5 @@
 	<xacro:arg name="use_laser_visual_mesh" default='false'/>
 	<xacro:arg name="use_lidar" default='true'/>
+	<xacro:arg name="enable_sensors" default='true'/>
 	<xacro:arg name="use_lift" default='true'/>
 	<xacro:property name="use_lift" value="$(arg use_lift)"/>
@@ -75,5 +76,5 @@
 		controllers_file="$(arg simulation_controllers)"
 	/>
-	<xacro:gazebo_sim_sensors robot_namespace="$(arg robot_namespace)" use_lidar="$(arg use_lidar)"/>
+	<xacro:gazebo_sim_sensors robot_namespace="$(arg robot_namespace)" use_lidar="$(arg use_lidar)" enable_sensors="$(arg enable_sensors)"/>
 	<xacro:mir_robot_ros2_control/>
 	<xacro:if value="${use_arms}">
