Commit message: fixed lift_controllers

File: mir_robot/mir_description/ros2_control/mir_robot.ros2_control.xacro (robot description, xacro)
@@ -24,4 +24,22 @@
         <state_interface name="effort"/>
       </joint>
+      <joint name="right_lift_joint">
+        <command_interface name="position">
+          <param name="min">-1</param>
+          <param name="max">1</param>
+        </command_interface>
+        <state_interface name="position"/>
+        <state_interface name="velocity"/>
+        <state_interface name="effort"/>
+      </joint>
+      <joint name="left_lift_joint">
+        <command_interface name="position">
+          <param name="min">-1</param>
+          <param name="max">1</param>
+        </command_interface>
+        <state_interface name="position"/>
+        <state_interface name="velocity"/>
+        <state_interface name="effort"/>
+      </joint>
     </ros2_control>
   </xacro:macro>

File: mir_robot/mir_description/urdf/general/plugins.gazebo.xacro (robot description, xacro)
@@ -4,5 +4,5 @@
 		<gazebo>
 			<plugin filename="libgz_ros2_control-system.so" name="gz_ros2_control::GazeboSimROS2ControlPlugin">
-				<parameters>$(find mir_description)/config/diffdrive_controller.yaml</parameters>
+				<parameters>$(find mir_description)/config/mur_controllers.yaml</parameters>
 				<ros>
 					<xacro:unless value="${robot_namespace == ''}">

File: mir_robot/mir_description/urdf/mir_600/mir_600_top_lift.urdf.xacro (robot description, xacro)
@@ -63,8 +63,8 @@
 			<type>transmission_interface/SimpleTransmission</type>
 			<joint name="left_lift_joint">
-			  <hardwareInterface>hardware_interface/VelocityJointInterface</hardwareInterface>
+			  <hardwareInterface>hardware_interface/PositionJointInterface</hardwareInterface>
 			</joint>
 			<actuator name="left_lift_joint_motor">
-			  <hardwareInterface>hardware_interface/VelocityJointInterface</hardwareInterface>
+			  <hardwareInterface>hardware_interface/PositionJointInterface</hardwareInterface>
 			  <mechanicalReduction>1</mechanicalReduction>
 			</actuator>
@@ -73,8 +73,8 @@
 			<type>transmission_interface/SimpleTransmission</type>
 			<joint name="right_lift_joint">
-			  <hardwareInterface>hardware_interface/VelocityJointInterface</hardwareInterface>
+			  <hardwareInterface>hardware_interface/PositionJointInterface</hardwareInterface>
 			</joint>
 			<actuator name="right_lift_joint_motor">
-			  <hardwareInterface>hardware_interface/VelocityJointInterface</hardwareInterface>
+			  <hardwareInterface>hardware_interface/PositionJointInterface</hardwareInterface>
 			  <mechanicalReduction>1</mechanicalReduction>
 			</actuator>

File: mir_robot/mir_description/urdf/mur_620.gazebo.xacro (robot description, xacro)
@@ -35,5 +35,5 @@
 	<xacro:include filename="$(find ur_description)/urdf/ur_macro.xacro"/>
 	<xacro:include filename="$(find ur_simulation_gz)/urdf/ur_gz.ros2_control.xacro" />
-	<!-- <xacro:include filename="$(find mir_description)/ros2_control/mir_robot.ros2_control.xacro" /> -->
+	<xacro:include filename="$(find mir_description)/ros2_control/mir_robot.ros2_control.xacro" />
 	<xacro:include filename="$(find mir_description)/urdf/mir_600/mir_600_top_lift.urdf.xacro" />
 	<!-- Include plugin xacros -->
@@ -47,5 +47,5 @@
 	<xacro:p3d_base_controller robot_namespace="$(arg robot_namespace)"/>
 	<xacro:gazebo_sim_sensors robot_namespace="$(arg robot_namespace)"/>
-	<!-- <xacro:mir_robot_ros2_control/> -->
+	<xacro:mir_robot_ros2_control/>
 	<!-- UR10_l -->
 	<xacro:ur_robot

Commit message: fixed material warnings

File: mir_robot/mir_description/ros2_control/mir_robot.ros2_control.xacro (robot description, xacro)
@@ -6,5 +6,5 @@
           <plugin>gz_ros2_control/GazeboSimSystem</plugin>
       </hardware>
-      <joint name="left_wheel_joint">
+      <!-- <joint name="left_wheel_joint">
         <command_interface name="velocity">
           <param name="min">-1</param>
@@ -23,5 +23,5 @@
         <state_interface name="velocity"/>
         <state_interface name="effort"/>
-      </joint>
+      </joint> -->
       <joint name="right_lift_joint">
         <command_interface name="position">

File: mir_robot/mir_description/urdf/include/mir_v1.urdf.xacro (robot description, xacro)
@@ -106,5 +106,10 @@
     </link>
     <gazebo reference="${prefix}${locationprefix}_caster_rotation_link">
-      <material>Gazebo/Grey</material>
+      <material>
+        <ambient>0.5 0.5 0.5 1.0</ambient> <!-- Adjust as needed -->
+        <diffuse>0.5 0.5 0.5 1.0</diffuse>
+        <specular>0.1 0.1 0.1 1.0</specular>
+        <emissive>0 0 0 1</emissive>
+      </material>
     </gazebo>
     <!-- caster wheel -->

File: mir_robot/mir_description/urdf/mir_600/mir_600.gazebo.xacro (robot description, xacro)
@@ -30,5 +30,10 @@
 		<!-- Set Gazebo material for the base -->
 		<gazebo reference="base_link">
-			<material>Gazebo/Grey</material>
+			<material>
+				<ambient>0.5 0.5 0.5 1.0</ambient> <!-- Adjust as needed -->
+				<diffuse>0.5 0.5 0.5 1.0</diffuse>
+				<specular>0.1 0.1 0.1 1.0</specular>
+				<emissive>0 0 0 1</emissive>
+			</material>
 		</gazebo>
 		<!-- Set gazebo material for the wheels -->

File: mir_robot/mir_description/urdf/mir_600/mir_600_top_lift.urdf.xacro (robot description, xacro)
@@ -21,5 +21,10 @@
 		</link>
 		<gazebo reference="left_lift_top">
-			<material>Gazebo/Grey</material>
+			      <material>
+					<ambient>0.5 0.5 0.5 1.0</ambient> <!-- Adjust as needed -->
+					<diffuse>0.5 0.5 0.5 1.0</diffuse>
+					<specular>0.1 0.1 0.1 1.0</specular>
+					<emissive>0 0 0 1</emissive>
+				</material>
 		</gazebo>
 		<joint name="left_lift_joint" type="prismatic">
@@ -30,4 +35,8 @@
 			<limit lower="0.0" upper="0.5" effort="1000000" velocity="1.0"/>
 			<axis xyz="0 0 1" />
+			<gazebo>
+				<plugin filename="gz_ros2_control-system" name="gz_ros2_control::GazeboSimROS2ControlPlugin"/>
+				<hardwareInterface>PositionJointInterface</hardwareInterface> <!-- or Effort/Velocity -->
+			</gazebo>
 		</joint>
         <link name="right_lift_top">
@@ -50,5 +59,10 @@
 		</link>
 		<gazebo reference="right_lift_top">
-			<material>Gazebo/Grey</material>
+			      <material>
+					<ambient>0.5 0.5 0.5 1.0</ambient> <!-- Adjust as needed -->
+					<diffuse>0.5 0.5 0.5 1.0</diffuse>
+					<specular>0.1 0.1 0.1 1.0</specular>
+					<emissive>0 0 0 1</emissive>
+				</material>
 		</gazebo>
 		<joint name="right_lift_joint" type="prismatic">
@@ -59,4 +73,8 @@
 			<limit lower="0.0" upper="0.5" effort="1000000" velocity="1.0"/>
 			<axis xyz="0 0 1" />
+			<gazebo>
+				<plugin filename="gz_ros2_control-system" name="gz_ros2_control::GazeboSimROS2ControlPlugin"/>
+				<hardwareInterface>PositionJointInterface</hardwareInterface> <!-- or Effort/Velocity -->
+			</gazebo>
 		</joint>
 		<transmission name="left_lift_transmission">

File: mir_robot/mir_description/urdf/mir_600/mir_600_top_module.urdf.xacro (robot description, xacro)
@@ -23,5 +23,10 @@
 		</link>
 		<gazebo reference="top_module">
-			<material>Gazebo/Grey</material>
+			      <material>
+					<ambient>0.5 0.5 0.5 1.0</ambient> <!-- Adjust as needed -->
+					<diffuse>0.5 0.5 0.5 1.0</diffuse>
+					<specular>0.1 0.1 0.1 1.0</specular>
+					<emissive>0 0 0 1</emissive>
+				</material>
 		</gazebo>
 		<joint name="top_module_joint" type="fixed">
@@ -50,5 +55,10 @@
 		</link>
 		<gazebo reference="left_lift_bottom">
-			<material>Gazebo/DarkGrey</material>
+			<material>
+				<ambient>0.3 0.3 0.3 1.0</ambient> <!-- Dark grey -->
+				<diffuse>0.3 0.3 0.3 1.0</diffuse>
+				<specular>0.1 0.1 0.1 1.0</specular>
+				<emissive>0 0 0 1</emissive>
+			</material>
 		</gazebo>
 		<joint name="left_lift_bottom_joint" type="fixed">
@@ -77,5 +87,10 @@
 		</link>
 		<gazebo reference="right_lift_bottom">
-			<material>Gazebo/DarkGrey</material>
+			    <material>
+					<ambient>0.3 0.3 0.3 1.0</ambient> <!-- Dark grey -->
+					<diffuse>0.3 0.3 0.3 1.0</diffuse>
+					<specular>0.1 0.1 0.1 1.0</specular>
+					<emissive>0 0 0 1</emissive>
+				</material>
 		</gazebo>
 		<joint name="right_lift_bottom_joint" type="fixed">

File: mir_robot/mir_description/urdf/mir_600/mir_600_wheels.gazebo.xacro (robot description, xacro)
@@ -3,13 +3,28 @@
 	<xacro:macro name="actuated_wheel_gazebo" params="locationprefix">
 		<gazebo reference="${locationprefix}_wheel_link">
-			<material>Gazebo/DarkGrey</material>
+			    <material>
+					<ambient>0.3 0.3 0.3 1.0</ambient> <!-- Dark grey -->
+					<diffuse>0.3 0.3 0.3 1.0</diffuse>
+					<specular>0.1 0.1 0.1 1.0</specular>
+					<emissive>0 0 0 1</emissive>
+				</material>
 		</gazebo>
 	</xacro:macro>
 	<xacro:macro name="caster_wheel_gazebo" params="locationprefix">
 		<gazebo reference="${locationprefix}_caster_rotation_link">
-			<material>Gazebo/Grey</material>
+			      <material>
+					<ambient>0.5 0.5 0.5 1.0</ambient> <!-- Adjust as needed -->
+					<diffuse>0.5 0.5 0.5 1.0</diffuse>
+					<specular>0.1 0.1 0.1 1.0</specular>
+					<emissive>0 0 0 1</emissive>
+				</material>
 		</gazebo>
 		<gazebo reference="${locationprefix}_caster_wheel_link">
-			<material>Gazebo/DarkGrey</material>
+			    <material>
+					<ambient>0.3 0.3 0.3 1.0</ambient> <!-- Dark grey -->
+					<diffuse>0.3 0.3 0.3 1.0</diffuse>
+					<specular>0.1 0.1 0.1 1.0</specular>
+					<emissive>0 0 0 1</emissive>
+				</material>
 		</gazebo>
 	</xacro:macro>

File: mir_robot/urdf/include/mir_v1.urdf.xacro (robot description, xacro)
@@ -106,5 +106,10 @@
     </link>
     <gazebo reference="${prefix}${locationprefix}_caster_rotation_link">
-      <material>Gazebo/Grey</material>
+            <material>
+              <ambient>0.5 0.5 0.5 1.0</ambient> <!-- Adjust as needed -->
+              <diffuse>0.5 0.5 0.5 1.0</diffuse>
+              <specular>0.1 0.1 0.1 1.0</specular>
+              <emissive>0 0 0 1</emissive>
+            </material>
     </gazebo>
     <!-- caster wheel -->

Commit message: feat: update URDF and launch files to enhance controller integration and simulation parameters

File: mir_robot/mir_description/ros2_control/mir_robot.ros2_control.xacro (robot description, xacro)
@@ -27,5 +27,5 @@
         <command_interface name="position">
           <param name="min">0</param>
-          <param name="max">1</param>
+          <param name="max">0.5</param>
         </command_interface>
         <state_interface name="position"/>
@@ -36,5 +36,5 @@
         <command_interface name="position">
           <param name="min">0</param>
-          <param name="max">1</param>
+          <param name="max">0.5</param>
         </command_interface>
         <state_interface name="position"/>

File: mir_robot/mir_description/urdf/general/plugins.gazebo.xacro (robot description, xacro)
@@ -1,14 +1,12 @@
 <?xml version="1.0"?>
 <robot xmlns:xacro="http://ros.org/wiki/xacro">
-	<xacro:macro name="controller_plugin_gazebo" params="robot_namespace">
+	<xacro:macro name="controller_plugin_gazebo" params="robot_namespace controllers_file">
 		<gazebo>
 			<plugin filename="libgz_ros2_control-system.so" name="gz_ros2_control::GazeboSimROS2ControlPlugin">
-				<parameters>$(find mir_description)/config/mur_controllers.yaml</parameters>
+				<parameters>${controllers_file}</parameters>
 				<ros>
 					<xacro:unless value="${robot_namespace == ''}">
-						<robotNamespace>${robot_namespace}</robotNamespace>
+						<namespace>${robot_namespace}</namespace>
 					</xacro:unless>
-					<controlPeriod>0.001</controlPeriod>
-					<legacyModeNS>true</legacyModeNS>
 				</ros>
 			</plugin>

File: mir_robot/mir_description/urdf/mir_600/mir_600_top_lift.urdf.xacro (robot description, xacro)
@@ -28,16 +28,11 @@
 				</material>
 		</gazebo>
-		<!-- for some reason prismatic joint dont work, so we use a continuous joint - this is a workaround and should be fixed -->
-		<joint name="left_lift_joint" type="continuous">
+		<joint name="left_lift_joint" type="prismatic">
 			<origin xyz="0.0 0.0 0.0" rpy="0 0 0" />
 			<parent link="left_lift_bottom" />
 			<child link="left_lift_top" />
 			<dynamics damping="1.0" friction="1.0"/>
-			<limit lower="-0.01" upper="1.0" effort="1000000" velocity="1.0"/>
-			<axis xyz="0 1 0" />
-			<gazebo>
-				<plugin filename="gz_ros2_control-system" name="gz_ros2_control::GazeboSimROS2ControlPlugin"/>
-				<hardwareInterface>PositionJointInterface</hardwareInterface> <!-- or Effort/Velocity -->
-			</gazebo>
+			<limit lower="0.0" upper="0.5" effort="1000000" velocity="0.5"/>
+			<axis xyz="0 0 1" />
 		</joint>
         <link name="right_lift_top">
@@ -67,15 +62,11 @@
 				</material>
 		</gazebo>
-		<joint name="right_lift_joint" type="continuous">
+		<joint name="right_lift_joint" type="prismatic">
 			<origin xyz="0.0 0.0 0.0" rpy="0 0 0" />
 			<parent link="right_lift_bottom" />
 			<child link="right_lift_top" />
 			<dynamics damping="1.0" friction="1.0"/>
-			<limit lower="-0.01" upper="0.5" effort="1000000" velocity="1.0"/>
+			<limit lower="0.0" upper="0.5" effort="1000000" velocity="0.5"/>
 			<axis xyz="0 0 1" />
-			<gazebo>
-				<plugin filename="gz_ros2_control-system" name="gz_ros2_control::GazeboSimROS2ControlPlugin"/>
-				<hardwareInterface>PositionJointInterface</hardwareInterface> <!-- or Effort/Velocity -->
-			</gazebo>
 		</joint>
 		<transmission name="left_lift_transmission">

File: mur_robot/mur_description/urdf/mur_620.gazebo.xacro (robot description, xacro)
@@ -25,5 +25,5 @@
 	<xacro:arg name="safety_pos_margin" default="0.15"/>
 	<xacro:arg name="safety_k_position" default="20"/>
-	<xacro:arg name="simulation_controllers" default="" />
+	<xacro:arg name="simulation_controllers" default="$(find mir_description)/config/mur_controllers.yaml" />
 	<!-- MiR600 base -->
 	<xacro:include filename="$(find mir_description)/urdf/mir_600/mir_600.urdf.xacro" />
@@ -42,5 +42,8 @@
 	<xacro:mir_600_gazebo tf_prefix="$(arg tf_prefix_mir)" robot_namespace="$(arg robot_namespace)"/>
 	<!-- Init the plugins that run the MiR in Gazebo -->
-	<xacro:controller_plugin_gazebo robot_namespace="$(arg robot_namespace)"/>
+	<xacro:controller_plugin_gazebo
+		robot_namespace="$(arg robot_namespace)"
+		controllers_file="$(arg simulation_controllers)"
+	/>
 	<xacro:p3d_base_controller robot_namespace="$(arg robot_namespace)"/>
 	<xacro:gazebo_sim_sensors robot_namespace="$(arg robot_namespace)"/>

Commit message: forward velocity controller

File: mir_robot/mir_description/ros2_control/mir_robot.ros2_control.xacro (robot description, xacro)
@@ -42,4 +42,36 @@
         <state_interface name="effort"/>
       </joint>
+      <joint name="fl_caster_rotation_joint">
+        <state_interface name="position"/>
+        <state_interface name="velocity"/>
+      </joint>
+      <joint name="fl_caster_wheel_joint">
+        <state_interface name="position"/>
+        <state_interface name="velocity"/>
+      </joint>
+      <joint name="fr_caster_rotation_joint">
+        <state_interface name="position"/>
+        <state_interface name="velocity"/>
+      </joint>
+      <joint name="fr_caster_wheel_joint">
+        <state_interface name="position"/>
+        <state_interface name="velocity"/>
+      </joint>
+      <joint name="bl_caster_rotation_joint">
+        <state_interface name="position"/>
+        <state_interface name="velocity"/>
+      </joint>
+      <joint name="bl_caster_wheel_joint">
+        <state_interface name="position"/>
+        <state_interface name="velocity"/>
+      </joint>
+      <joint name="br_caster_rotation_joint">
+        <state_interface name="position"/>
+        <state_interface name="velocity"/>
+      </joint>
+      <joint name="br_caster_wheel_joint">
+        <state_interface name="position"/>
+        <state_interface name="velocity"/>
+      </joint>
     </ros2_control>
   </xacro:macro>
