Commit message: hardware

File: mur_robot/mur_description/urdf/mur_620.gazebo.xacro (robot description, xacro)
@@ -90,5 +90,5 @@
 			force_abs_paths="true"
 			>
-			<origin xyz="0 0 0" rpy="$(arg ur_l_rpy)" />          <!-- position robot in the world -->
+			<origin xyz="$(arg ur_l_xyz)" rpy="$(arg ur_l_rpy)" />          <!-- position robot in the world -->
 		</xacro:ur_robot>
 		<xacro:ur_robot
@@ -105,5 +105,5 @@
 			force_abs_paths="true"
 			>
-			<origin xyz="0 0 0" rpy="$(arg ur_r_rpy)" />          <!-- position robot in the world -->
+			<origin xyz="$(arg ur_r_xyz)" rpy="$(arg ur_r_rpy)" />          <!-- position robot in the world -->
 		</xacro:ur_robot>
 		<xacro:ur_ros2_control
