Commit message: Add ewellix dual state to joint state bridge and update launch configurations
- Added `ewellix_dual_state_to_joint_state.py` script to convert Ewellix dual state messages to ROS JointState messages.
- Updated `CMakeLists.txt` to install the new script.
- Modified `mur_robot_profiles.yaml` to include custom home positions for shoulder pan joints.
- Created a new RViz configuration file for the mur620d robot.
- Updated launch files to integrate the new dual state bridge and adjusted parameters for integrated controllers.
- Enhanced the UR MoveIt launch file to accept custom shoulder pan angles for home positions.
- Updated SRDF Xacro file to use the new custom shoulder pan angles in the Home_custom state.
- Adjusted the `start_mur620_hardware_logged.sh` script to include the new state bridge and related scripts.

File: mur_robot/mur_moveit_config/srdf/mur620.srdf.xacro (robot description, xacro)
@@ -8,4 +8,6 @@
     <xacro:arg name="prefix" default=""/>
     <xacro:arg name="virtual_joint_parent_frame" default="world"/>
+    <xacro:arg name="home_custom_l_shoulder_pan" default="0.0"/>
+    <xacro:arg name="home_custom_r_shoulder_pan" default="0.0"/>
     <virtual_joint
         name="fixed_base"
@@ -119,5 +121,5 @@
         <joint name="$(arg prefix)_l/elbow_joint" value="-1.57079632679 "/>
         <joint name="$(arg prefix)_l/shoulder_lift_joint" value="-1.57079632679 "/>
-        <joint name="$(arg prefix)_l/shoulder_pan_joint" value="-0.0"/>
+        <joint name="$(arg prefix)_l/shoulder_pan_joint" value="$(arg home_custom_l_shoulder_pan)"/>
         <joint name="$(arg prefix)_l/wrist_1_joint" value="-1.57079632679 "/>
         <joint name="$(arg prefix)_l/wrist_2_joint" value="1.57079632679 "/>
@@ -127,5 +129,5 @@
         <joint name="$(arg prefix)_r/elbow_joint" value="1.57079632679"/>
         <joint name="$(arg prefix)_r/shoulder_lift_joint" value="-1.57079632679"/>
-        <joint name="$(arg prefix)_r/shoulder_pan_joint" value="-0.0"/>
+        <joint name="$(arg prefix)_r/shoulder_pan_joint" value="$(arg home_custom_r_shoulder_pan)"/>
         <joint name="$(arg prefix)_r/wrist_1_joint" value="-1.57079632679"/>
         <joint name="$(arg prefix)_r/wrist_2_joint" value="-1.57079632679"/>
