Commit message: Refactor launch and configuration for lift functionality in MuR620
- Updated README.md to clarify build instructions for the `ewellix_driver` package.
- Modified `mur_620.launch.py` to include remapping for joint states and added parameters for robot geometry and lift usage.
- Enhanced `ur_moveit.launch.py` to conditionally include lift controllers based on the `use_lift` argument.
- Adjusted `mur620.srdf.xacro` to conditionally include lift joints and collision settings based on the `use_lift` argument.
- Improved `start_mur620_hardware_logged.sh` to handle lift configuration based on profiles and command-line arguments.

File: mur_robot/mur_moveit_config/srdf/mur620.srdf.xacro (robot description, xacro)
@@ -7,4 +7,5 @@
         xmlns:xacro="http://www.ros.org/wiki/xacro">
     <xacro:arg name="prefix" default=""/>
+    <xacro:arg name="use_lift" default="true"/>
     <xacro:arg name="virtual_joint_parent_frame" default="world"/>
     <xacro:arg name="home_custom_l_shoulder_pan" default="0.0"/>
@@ -62,4 +63,5 @@
         <joint name="$(arg prefix)_r/flange-tool0"/>
     </group>
+    <xacro:if value="$(arg use_lift)">
 	<group name="UR_arm_lift_l">
 		<joint name="left_lift_joint"/>
@@ -86,6 +88,9 @@
         <joint name="$(arg prefix)_r/flange-tool0"/>
     </group>
+    </xacro:if>
 	<group name="UR_arm_all">
-		<joint name="left_lift_joint"/>
+        <xacro:if value="$(arg use_lift)">
+		    <joint name="left_lift_joint"/>
+        </xacro:if>
 		<joint name="$(arg prefix)_l/base_link-base_link_inertia"/>
         <joint name="$(arg prefix)_l/shoulder_pan_joint"/>
@@ -97,5 +102,7 @@
         <joint name="$(arg prefix)_l/wrist_3-flange"/>
         <joint name="$(arg prefix)_l/flange-tool0"/>
-        <joint name="right_lift_joint"/>
+        <xacro:if value="$(arg use_lift)">
+            <joint name="right_lift_joint"/>
+        </xacro:if>
 		<joint name="$(arg prefix)_r/base_link-base_link_inertia"/>
         <joint name="$(arg prefix)_r/shoulder_pan_joint"/>
@@ -259,8 +266,6 @@
     <disable_collisions link1="$(arg prefix)_l/base_link_inertia" link2="front_laser_link" reason="Never"/>
     <disable_collisions link1="$(arg prefix)_l/base_link_inertia" link2="left_lift_bottom" reason="Never"/>
-    <disable_collisions link1="$(arg prefix)_l/base_link_inertia" link2="left_lift_top" reason="Adjacent"/>
     <disable_collisions link1="$(arg prefix)_l/base_link_inertia" link2="left_wheel_link" reason="Never"/>
     <disable_collisions link1="$(arg prefix)_l/base_link_inertia" link2="right_lift_bottom" reason="Never"/>
-    <disable_collisions link1="$(arg prefix)_l/base_link_inertia" link2="right_lift_top" reason="Never"/>
     <disable_collisions link1="$(arg prefix)_l/base_link_inertia" link2="right_wheel_link" reason="Never"/>
     <disable_collisions link1="$(arg prefix)_l/base_link_inertia" link2="top_module" reason="Never"/>
@@ -290,18 +295,8 @@
     <disable_collisions link1="$(arg prefix)_l/shoulder_link" link2="front_laser_link" reason="Never"/>
     <disable_collisions link1="$(arg prefix)_l/shoulder_link" link2="left_lift_bottom" reason="Never"/>
-    <disable_collisions link1="$(arg prefix)_l/shoulder_link" link2="left_lift_top" reason="Never"/>
     <disable_collisions link1="$(arg prefix)_l/shoulder_link" link2="left_wheel_link" reason="Never"/>
     <disable_collisions link1="$(arg prefix)_l/shoulder_link" link2="right_lift_bottom" reason="Never"/>
-    <disable_collisions link1="$(arg prefix)_l/shoulder_link" link2="right_lift_top" reason="Never"/>
     <disable_collisions link1="$(arg prefix)_l/shoulder_link" link2="right_wheel_link" reason="Never"/>
     <disable_collisions link1="$(arg prefix)_l/shoulder_link" link2="top_module" reason="Never"/>
-    <disable_collisions link1="$(arg prefix)_l/tcp" link2="$(arg prefix)_l/wrist_1_link" reason="Never"/>
-    <disable_collisions link1="$(arg prefix)_l/tcp" link2="$(arg prefix)_l/wrist_2_link" reason="Never"/>
-    <disable_collisions link1="$(arg prefix)_l/tcp" link2="$(arg prefix)_l/wrist_3_link" reason="Adjacent"/>
-    <disable_collisions link1="$(arg prefix)_l/tcp" link2="back_laser_link" reason="Never"/>
-    <disable_collisions link1="$(arg prefix)_l/tcp" link2="bl_caster_rotation_link" reason="Never"/>
-    <disable_collisions link1="$(arg prefix)_l/tcp" link2="bl_caster_wheel_link" reason="Never"/>
-    <disable_collisions link1="$(arg prefix)_l/tcp" link2="br_caster_rotation_link" reason="Never"/>
-    <disable_collisions link1="$(arg prefix)_l/tcp" link2="br_caster_wheel_link" reason="Never"/>
     <disable_collisions link1="$(arg prefix)_l/upper_arm_link" link2="back_laser_link" reason="Never"/>
     <disable_collisions link1="$(arg prefix)_l/upper_arm_link" link2="base_link" reason="Never"/>
@@ -325,5 +320,4 @@
     <disable_collisions link1="$(arg prefix)_l/wrist_1_link" link2="br_caster_rotation_link" reason="Never"/>
     <disable_collisions link1="$(arg prefix)_l/wrist_1_link" link2="br_caster_wheel_link" reason="Never"/>
-    <disable_collisions link1="$(arg prefix)_l/wrist_1_link" link2="left_lift_top" reason="Never"/>
     <disable_collisions link1="$(arg prefix)_l/wrist_1_link" link2="right_wheel_link" reason="Never"/>
     <disable_collisions link1="$(arg prefix)_l/wrist_2_link" link2="$(arg prefix)_l/wrist_3_link" reason="Adjacent"/>
@@ -354,8 +348,6 @@
     <disable_collisions link1="$(arg prefix)_r/base_link_inertia" link2="front_laser_link" reason="Never"/>
     <disable_collisions link1="$(arg prefix)_r/base_link_inertia" link2="left_lift_bottom" reason="Never"/>
-    <disable_collisions link1="$(arg prefix)_r/base_link_inertia" link2="left_lift_top" reason="Never"/>
     <disable_collisions link1="$(arg prefix)_r/base_link_inertia" link2="left_wheel_link" reason="Never"/>
     <disable_collisions link1="$(arg prefix)_r/base_link_inertia" link2="right_lift_bottom" reason="Never"/>
-    <disable_collisions link1="$(arg prefix)_r/base_link_inertia" link2="right_lift_top" reason="Adjacent"/>
     <disable_collisions link1="$(arg prefix)_r/base_link_inertia" link2="right_wheel_link" reason="Never"/>
     <disable_collisions link1="$(arg prefix)_r/base_link_inertia" link2="top_module" reason="Never"/>
@@ -383,17 +375,8 @@
     <disable_collisions link1="$(arg prefix)_r/shoulder_link" link2="front_laser_link" reason="Never"/>
     <disable_collisions link1="$(arg prefix)_r/shoulder_link" link2="left_lift_bottom" reason="Never"/>
-    <disable_collisions link1="$(arg prefix)_r/shoulder_link" link2="left_lift_top" reason="Never"/>
     <disable_collisions link1="$(arg prefix)_r/shoulder_link" link2="left_wheel_link" reason="Never"/>
     <disable_collisions link1="$(arg prefix)_r/shoulder_link" link2="right_lift_bottom" reason="Never"/>
-    <disable_collisions link1="$(arg prefix)_r/shoulder_link" link2="right_lift_top" reason="Never"/>
     <disable_collisions link1="$(arg prefix)_r/shoulder_link" link2="right_wheel_link" reason="Never"/>
     <disable_collisions link1="$(arg prefix)_r/shoulder_link" link2="top_module" reason="Never"/>
-    <disable_collisions link1="$(arg prefix)_r/tcp" link2="$(arg prefix)_r/wrist_1_link" reason="Never"/>
-    <disable_collisions link1="$(arg prefix)_r/tcp" link2="$(arg prefix)_r/wrist_2_link" reason="Never"/>
-    <disable_collisions link1="$(arg prefix)_r/tcp" link2="$(arg prefix)_r/wrist_3_link" reason="Adjacent"/>
-    <disable_collisions link1="$(arg prefix)_r/tcp" link2="back_laser_link" reason="Never"/>
-    <disable_collisions link1="$(arg prefix)_r/tcp" link2="bl_caster_rotation_link" reason="Never"/>
-    <disable_collisions link1="$(arg prefix)_r/tcp" link2="bl_caster_wheel_link" reason="Never"/>
-    <disable_collisions link1="$(arg prefix)_r/tcp" link2="br_caster_wheel_link" reason="Never"/>
     <disable_collisions link1="$(arg prefix)_r/upper_arm_link" link2="back_laser_link" reason="Never"/>
     <disable_collisions link1="$(arg prefix)_r/upper_arm_link" link2="base_link" reason="Never"/>
@@ -417,5 +400,4 @@
     <disable_collisions link1="$(arg prefix)_r/wrist_1_link" link2="br_caster_rotation_link" reason="Never"/>
     <disable_collisions link1="$(arg prefix)_r/wrist_1_link" link2="br_caster_wheel_link" reason="Never"/>
-    <disable_collisions link1="$(arg prefix)_r/wrist_1_link" link2="right_lift_top" reason="Never"/>
     <disable_collisions link1="$(arg prefix)_r/wrist_2_link" link2="$(arg prefix)_r/wrist_3_link" reason="Adjacent"/>
     <disable_collisions link1="$(arg prefix)_r/wrist_2_link" link2="back_laser_link" reason="Never"/>
@@ -442,8 +424,6 @@
     <disable_collisions link1="back_laser_link" link2="front_laser_link" reason="Never"/>
     <disable_collisions link1="back_laser_link" link2="left_lift_bottom" reason="Never"/>
-    <disable_collisions link1="back_laser_link" link2="left_lift_top" reason="Never"/>
     <disable_collisions link1="back_laser_link" link2="left_wheel_link" reason="Never"/>
     <disable_collisions link1="back_laser_link" link2="right_lift_bottom" reason="Never"/>
-    <disable_collisions link1="back_laser_link" link2="right_lift_top" reason="Never"/>
     <disable_collisions link1="back_laser_link" link2="right_wheel_link" reason="Never"/>
     <disable_collisions link1="back_laser_link" link2="top_module" reason="Never"/>
@@ -459,8 +439,6 @@
     <disable_collisions link1="base_link" link2="front_laser_link" reason="Adjacent"/>
     <disable_collisions link1="base_link" link2="left_lift_bottom" reason="Never"/>
-    <disable_collisions link1="base_link" link2="left_lift_top" reason="Never"/>
     <disable_collisions link1="base_link" link2="left_wheel_link" reason="Adjacent"/>
     <disable_collisions link1="base_link" link2="right_lift_bottom" reason="Never"/>
-    <disable_collisions link1="base_link" link2="right_lift_top" reason="Never"/>
     <disable_collisions link1="base_link" link2="right_wheel_link" reason="Adjacent"/>
     <disable_collisions link1="base_link" link2="top_module" reason="Adjacent"/>
@@ -475,8 +453,6 @@
     <disable_collisions link1="bl_caster_rotation_link" link2="front_laser_link" reason="Never"/>
     <disable_collisions link1="bl_caster_rotation_link" link2="left_lift_bottom" reason="Never"/>
-    <disable_collisions link1="bl_caster_rotation_link" link2="left_lift_top" reason="Never"/>
     <disable_collisions link1="bl_caster_rotation_link" link2="left_wheel_link" reason="Never"/>
     <disable_collisions link1="bl_caster_rotation_link" link2="right_lift_bottom" reason="Never"/>
-    <disable_collisions link1="bl_caster_rotation_link" link2="right_lift_top" reason="Never"/>
     <disable_collisions link1="bl_caster_rotation_link" link2="right_wheel_link" reason="Never"/>
     <disable_collisions link1="bl_caster_rotation_link" link2="top_module" reason="Never"/>
@@ -490,8 +466,6 @@
     <disable_collisions link1="bl_caster_wheel_link" link2="front_laser_link" reason="Never"/>
     <disable_collisions link1="bl_caster_wheel_link" link2="left_lift_bottom" reason="Never"/>
-    <disable_collisions link1="bl_caster_wheel_link" link2="left_lift_top" reason="Never"/>
     <disable_collisions link1="bl_caster_wheel_link" link2="left_wheel_link" reason="Never"/>
     <disable_collisions link1="bl_caster_wheel_link" link2="right_lift_bottom" reason="Never"/>
-    <disable_collisions link1="bl_caster_wheel_link" link2="right_lift_top" reason="Never"/>
     <disable_collisions link1="bl_caster_wheel_link" link2="right_wheel_link" reason="Never"/>
     <disable_collisions link1="bl_caster_wheel_link" link2="top_module" reason="Never"/>
@@ -504,8 +478,6 @@
     <disable_collisions link1="br_caster_rotation_link" link2="front_laser_link" reason="Never"/>
     <disable_collisions link1="br_caster_rotation_link" link2="left_lift_bottom" reason="Never"/>
-    <disable_collisions link1="br_caster_rotation_link" link2="left_lift_top" reason="Never"/>
     <disable_collisions link1="br_caster_rotation_link" link2="left_wheel_link" reason="Never"/>
     <disable_collisions link1="br_caster_rotation_link" link2="right_lift_bottom" reason="Never"/>
-    <disable_collisions link1="br_caster_rotation_link" link2="right_lift_top" reason="Never"/>
     <disable_collisions link1="br_caster_rotation_link" link2="right_wheel_link" reason="Never"/>
     <disable_collisions link1="br_caster_rotation_link" link2="top_module" reason="Never"/>
@@ -517,8 +489,6 @@
     <disable_collisions link1="br_caster_wheel_link" link2="front_laser_link" reason="Never"/>
     <disable_collisions link1="br_caster_wheel_link" link2="left_lift_bottom" reason="Never"/>
-    <disable_collisions link1="br_caster_wheel_link" link2="left_lift_top" reason="Never"/>
     <disable_collisions link1="br_caster_wheel_link" link2="left_wheel_link" reason="Never"/>
     <disable_collisions link1="br_caster_wheel_link" link2="right_lift_bottom" reason="Never"/>
-    <disable_collisions link1="br_caster_wheel_link" link2="right_lift_top" reason="Never"/>
     <disable_collisions link1="br_caster_wheel_link" link2="right_wheel_link" reason="Never"/>
     <disable_collisions link1="br_caster_wheel_link" link2="top_module" reason="Never"/>
@@ -529,8 +499,6 @@
     <disable_collisions link1="camera_link" link2="front_laser_link" reason="Never"/>
     <disable_collisions link1="camera_link" link2="left_lift_bottom" reason="Never"/>
-    <disable_collisions link1="camera_link" link2="left_lift_top" reason="Never"/>
     <disable_collisions link1="camera_link" link2="left_wheel_link" reason="Never"/>
     <disable_collisions link1="camera_link" link2="right_lift_bottom" reason="Never"/>
-    <disable_collisions link1="camera_link" link2="right_lift_top" reason="Never"/>
     <disable_collisions link1="camera_link" link2="right_wheel_link" reason="Never"/>
     <disable_collisions link1="camera_link" link2="top_module" reason="Never"/>
@@ -540,8 +508,6 @@
     <disable_collisions link1="fl_caster_rotation_link" link2="front_laser_link" reason="Never"/>
     <disable_collisions link1="fl_caster_rotation_link" link2="left_lift_bottom" reason="Never"/>
-    <disable_collisions link1="fl_caster_rotation_link" link2="left_lift_top" reason="Never"/>
     <disable_collisions link1="fl_caster_rotation_link" link2="left_wheel_link" reason="Never"/>
     <disable_collisions link1="fl_caster_rotation_link" link2="right_lift_bottom" reason="Never"/>
-    <disable_collisions link1="fl_caster_rotation_link" link2="right_lift_top" reason="Never"/>
     <disable_collisions link1="fl_caster_rotation_link" link2="right_wheel_link" reason="Never"/>
     <disable_collisions link1="fl_caster_rotation_link" link2="top_module" reason="Never"/>
@@ -550,8 +516,6 @@
     <disable_collisions link1="fl_caster_wheel_link" link2="front_laser_link" reason="Never"/>
     <disable_collisions link1="fl_caster_wheel_link" link2="left_lift_bottom" reason="Never"/>
-    <disable_collisions link1="fl_caster_wheel_link" link2="left_lift_top" reason="Never"/>
     <disable_collisions link1="fl_caster_wheel_link" link2="left_wheel_link" reason="Never"/>
     <disable_collisions link1="fl_caster_wheel_link" link2="right_lift_bottom" reason="Never"/>
-    <disable_collisions link1="fl_caster_wheel_link" link2="right_lift_top" reason="Never"/>
     <disable_collisions link1="fl_caster_wheel_link" link2="right_wheel_link" reason="Never"/>
     <disable_collisions link1="fl_caster_wheel_link" link2="top_module" reason="Never"/>
@@ -559,31 +523,67 @@
     <disable_collisions link1="fr_caster_rotation_link" link2="front_laser_link" reason="Never"/>
     <disable_collisions link1="fr_caster_rotation_link" link2="left_lift_bottom" reason="Never"/>
-    <disable_collisions link1="fr_caster_rotation_link" link2="left_lift_top" reason="Never"/>
     <disable_collisions link1="fr_caster_rotation_link" link2="left_wheel_link" reason="Never"/>
     <disable_collisions link1="fr_caster_rotation_link" link2="right_lift_bottom" reason="Never"/>
-    <disable_collisions link1="fr_caster_rotation_link" link2="right_lift_top" reason="Never"/>
     <disable_collisions link1="fr_caster_rotation_link" link2="right_wheel_link" reason="Never"/>
     <disable_collisions link1="fr_caster_rotation_link" link2="top_module" reason="Never"/>
     <disable_collisions link1="fr_caster_wheel_link" link2="front_laser_link" reason="Never"/>
     <disable_collisions link1="fr_caster_wheel_link" link2="left_lift_bottom" reason="Never"/>
-    <disable_collisions link1="fr_caster_wheel_link" link2="left_lift_top" reason="Never"/>
     <disable_collisions link1="fr_caster_wheel_link" link2="left_wheel_link" reason="Never"/>
     <disable_collisions link1="fr_caster_wheel_link" link2="right_lift_bottom" reason="Never"/>
-    <disable_collisions link1="fr_caster_wheel_link" link2="right_lift_top" reason="Never"/>
     <disable_collisions link1="fr_caster_wheel_link" link2="right_wheel_link" reason="Never"/>
     <disable_collisions link1="fr_caster_wheel_link" link2="top_module" reason="Never"/>
     <disable_collisions link1="front_laser_link" link2="left_lift_bottom" reason="Never"/>
-    <disable_collisions link1="front_laser_link" link2="left_lift_top" reason="Never"/>
     <disable_collisions link1="front_laser_link" link2="left_wheel_link" reason="Never"/>
     <disable_collisions link1="front_laser_link" link2="right_lift_bottom" reason="Never"/>
-    <disable_collisions link1="front_laser_link" link2="right_lift_top" reason="Never"/>
     <disable_collisions link1="front_laser_link" link2="right_wheel_link" reason="Never"/>
     <disable_collisions link1="front_laser_link" link2="top_module" reason="Never"/>
-    <disable_collisions link1="left_lift_bottom" link2="left_lift_top" reason="Adjacent"/>
     <disable_collisions link1="left_lift_bottom" link2="left_wheel_link" reason="Never"/>
     <disable_collisions link1="left_lift_bottom" link2="right_lift_bottom" reason="Never"/>
-    <disable_collisions link1="left_lift_bottom" link2="right_lift_top" reason="Never"/>
     <disable_collisions link1="left_lift_bottom" link2="right_wheel_link" reason="Never"/>
     <disable_collisions link1="left_lift_bottom" link2="top_module" reason="Adjacent"/>
+    <disable_collisions link1="left_wheel_link" link2="right_lift_bottom" reason="Never"/>
+    <disable_collisions link1="left_wheel_link" link2="right_wheel_link" reason="Never"/>
+    <disable_collisions link1="left_wheel_link" link2="top_module" reason="Never"/>
+    <disable_collisions link1="right_lift_bottom" link2="right_wheel_link" reason="Never"/>
+    <disable_collisions link1="right_lift_bottom" link2="top_module" reason="Adjacent"/>
+    <disable_collisions link1="right_wheel_link" link2="top_module" reason="Never"/>
+    <!-- Lift-top links are absent on MuR620a/b. -->
+    <xacro:if value="$(arg use_lift)">
+    <disable_collisions link1="$(arg prefix)_l/base_link_inertia" link2="left_lift_top" reason="Adjacent"/>
+    <disable_collisions link1="$(arg prefix)_l/base_link_inertia" link2="right_lift_top" reason="Never"/>
+    <disable_collisions link1="$(arg prefix)_l/shoulder_link" link2="left_lift_top" reason="Never"/>
+    <disable_collisions link1="$(arg prefix)_l/shoulder_link" link2="right_lift_top" reason="Never"/>
+    <disable_collisions link1="$(arg prefix)_l/wrist_1_link" link2="left_lift_top" reason="Never"/>
+    <disable_collisions link1="$(arg prefix)_r/base_link_inertia" link2="left_lift_top" reason="Never"/>
+    <disable_collisions link1="$(arg prefix)_r/base_link_inertia" link2="right_lift_top" reason="Adjacent"/>
+    <disable_collisions link1="$(arg prefix)_r/shoulder_link" link2="left_lift_top" reason="Never"/>
+    <disable_collisions link1="$(arg prefix)_r/shoulder_link" link2="right_lift_top" reason="Never"/>
+    <disable_collisions link1="$(arg prefix)_r/wrist_1_link" link2="right_lift_top" reason="Never"/>
+    <disable_collisions link1="back_laser_link" link2="left_lift_top" reason="Never"/>
+    <disable_collisions link1="back_laser_link" link2="right_lift_top" reason="Never"/>
+    <disable_collisions link1="base_link" link2="left_lift_top" reason="Never"/>
+    <disable_collisions link1="base_link" link2="right_lift_top" reason="Never"/>
+    <disable_collisions link1="bl_caster_rotation_link" link2="left_lift_top" reason="Never"/>
+    <disable_collisions link1="bl_caster_rotation_link" link2="right_lift_top" reason="Never"/>
+    <disable_collisions link1="bl_caster_wheel_link" link2="left_lift_top" reason="Never"/>
+    <disable_collisions link1="bl_caster_wheel_link" link2="right_lift_top" reason="Never"/>
+    <disable_collisions link1="br_caster_rotation_link" link2="left_lift_top" reason="Never"/>
+    <disable_collisions link1="br_caster_rotation_link" link2="right_lift_top" reason="Never"/>
+    <disable_collisions link1="br_caster_wheel_link" link2="left_lift_top" reason="Never"/>
+    <disable_collisions link1="br_caster_wheel_link" link2="right_lift_top" reason="Never"/>
+    <disable_collisions link1="camera_link" link2="left_lift_top" reason="Never"/>
+    <disable_collisions link1="camera_link" link2="right_lift_top" reason="Never"/>
+    <disable_collisions link1="fl_caster_rotation_link" link2="left_lift_top" reason="Never"/>
+    <disable_collisions link1="fl_caster_rotation_link" link2="right_lift_top" reason="Never"/>
+    <disable_collisions link1="fl_caster_wheel_link" link2="left_lift_top" reason="Never"/>
+    <disable_collisions link1="fl_caster_wheel_link" link2="right_lift_top" reason="Never"/>
+    <disable_collisions link1="fr_caster_rotation_link" link2="left_lift_top" reason="Never"/>
+    <disable_collisions link1="fr_caster_rotation_link" link2="right_lift_top" reason="Never"/>
+    <disable_collisions link1="fr_caster_wheel_link" link2="left_lift_top" reason="Never"/>
+    <disable_collisions link1="fr_caster_wheel_link" link2="right_lift_top" reason="Never"/>
+    <disable_collisions link1="front_laser_link" link2="left_lift_top" reason="Never"/>
+    <disable_collisions link1="front_laser_link" link2="right_lift_top" reason="Never"/>
+    <disable_collisions link1="left_lift_bottom" link2="left_lift_top" reason="Adjacent"/>
+    <disable_collisions link1="left_lift_bottom" link2="right_lift_top" reason="Never"/>
     <disable_collisions link1="left_lift_top" link2="left_wheel_link" reason="Never"/>
     <disable_collisions link1="left_lift_top" link2="right_lift_bottom" reason="Never"/>
@@ -591,13 +591,8 @@
     <disable_collisions link1="left_lift_top" link2="right_wheel_link" reason="Never"/>
     <disable_collisions link1="left_lift_top" link2="top_module" reason="Never"/>
-    <disable_collisions link1="left_wheel_link" link2="right_lift_bottom" reason="Never"/>
     <disable_collisions link1="left_wheel_link" link2="right_lift_top" reason="Never"/>
-    <disable_collisions link1="left_wheel_link" link2="right_wheel_link" reason="Never"/>
-    <disable_collisions link1="left_wheel_link" link2="top_module" reason="Never"/>
     <disable_collisions link1="right_lift_bottom" link2="right_lift_top" reason="Adjacent"/>
-    <disable_collisions link1="right_lift_bottom" link2="right_wheel_link" reason="Never"/>
-    <disable_collisions link1="right_lift_bottom" link2="top_module" reason="Adjacent"/>
     <disable_collisions link1="right_lift_top" link2="right_wheel_link" reason="Never"/>
     <disable_collisions link1="right_lift_top" link2="top_module" reason="Never"/>
-    <disable_collisions link1="right_wheel_link" link2="top_module" reason="Never"/>
+    </xacro:if>
 </robot>
